Commit message: slow brakeing is back, but at least we are running straight af

File: ros/src/leremix_control/urdf/LeRemix.hardware.xacro (robot description, xacro)
@@ -12,15 +12,15 @@
             <param name="publish_if_unchanged">true</param>
         </hardware>
-        <joint name="back_motor_rotation">
+        <joint name="wheel3_rotation">
             <command_interface name="velocity"/>
             <state_interface name="position"/>
             <state_interface name="velocity"/>
         </joint>
-        <joint name="left_motor_rotation">
+        <joint name="wheel1_rotation">
             <command_interface name="velocity"/>
             <state_interface name="position"/>
             <state_interface name="velocity"/>
         </joint>
-        <joint name="right_motor_rotation">
+        <joint name="wheel2_rotation">
             <command_interface name="velocity"/>
             <state_interface name="position"/>

File: ros/src/leremix_gazebo/urdf/initial_positions.xacro (robot description, xacro)
@@ -18,7 +18,7 @@
       <initial_joint_position name="camera_tilt">0.0</initial_joint_position> <!-- Camera: servo 11, relaxed (2048 counts = center) -->
       <!-- Motor initial positions (for reference) -->
-      <initial_joint_position name="back_motor_rotation">0.0</initial_joint_position>
-      <initial_joint_position name="left_motor_rotation">0.0</initial_joint_position>
-      <initial_joint_position name="right_motor_rotation">0.0</initial_joint_position>
+      <initial_joint_position name="wheel1_rotation">0.0</initial_joint_position>
+      <initial_joint_position name="wheel2_rotation">0.0</initial_joint_position>
+      <initial_joint_position name="wheel3_rotation">0.0</initial_joint_position>
     </plugin>
   </gazebo>
