Commit message: finally fixed urdf joints

File: ros/src/leremix_description/urdf/LeRemix.xacro (robot description, xacro)
@@ -4,12 +4,12 @@
 <link name="base_link">
   <inertial>
-    <origin xyz="-0.006995872672132321 0.00016351719531705557 -0.0020614117608215563" rpy="0 0 0"/>
-    <mass value="1.5793453539076083"/>
-    <inertia ixx="0.00541" iyy="0.005179" izz="0.010582" ixy="-3e-06" iyz="0.0" ixz="0.0"/>
+    <origin xyz="3.340802284881761e-05 0.0062553486303636415 0.0025000000000001423" rpy="0 0 0"/>
+    <mass value="1.5793453539076086"/>
+    <inertia ixx="0.005179" iyy="0.00541" izz="0.010582" ixy="3e-06" iyz="-0.0" ixz="0.0"/>
   </inertial>
   <visual>
     <origin xyz="0 0 0" rpy="0 0 0"/>
     <geometry>
-      <mesh filename="file://$(find LeRemix_description)/meshes/base_link.stl" scale="0.001 0.001 0.001"/>
+      <mesh filename="file://$(find leremix_description)/meshes/base_link.stl" scale="0.001 0.001 0.001"/>
     </geometry>
     <material name="silver"/>
@@ -18,5 +18,5 @@
     <origin xyz="0 0 0" rpy="0 0 0"/>
     <geometry>
-      <mesh filename="file://$(find LeRemix_description)/meshes/base_link.stl" scale="0.001 0.001 0.001"/>
+      <mesh filename="file://$(find leremix_description)/meshes/base_link.stl" scale="0.001 0.001 0.001"/>
     </geometry>
   </collision>
@@ -24,19 +24,79 @@
 <link name="arm_base_rotation_servo_1">
   <inertial>
-    <origin xyz="0.019999508147657045 0.010249860525163957 0.01602665316389948" rpy="0 0 0"/>
+    <origin xyz="0.010249751352689343 -0.01999903218942549 0.016027064924724457" rpy="0 0 0"/>
     <mass value="0.2843033831904074"/>
-    <inertia ixx="4e-05" iyy="7.3e-05" izz="6.2e-05" ixy="0.0" iyz="0.0" ixz="-1e-06"/>
-  </inertial>
-  <visual>
-    <origin xyz="-0.043607 0.01012 -0.080739" rpy="0 0 0"/>
-    <geometry>
-      <mesh filename="file://$(find LeRemix_description)/meshes/arm_base_rotation_servo_1.stl" scale="0.001 0.001 0.001"/>
-    </geometry>
-    <material name="silver"/>
-  </visual>
-  <collision>
-    <origin xyz="-0.043607 0.01012 -0.080739" rpy="0 0 0"/>
-    <geometry>
-      <mesh filename="file://$(find LeRemix_description)/meshes/arm_base_rotation_servo_1.stl" scale="0.001 0.001 0.001"/>
+    <inertia ixx="7.3e-05" iyy="4e-05" izz="6.2e-05" ixy="-0.0" iyz="1e-06" ixz="0.0"/>
+  </inertial>
+  <visual>
+    <origin xyz="0.01025 0.044348 -0.0853" rpy="0 0 0"/>
+    <geometry>
+      <mesh filename="file://$(find leremix_description)/meshes/arm_base_rotation_servo_1.stl" scale="0.001 0.001 0.001"/>
+    </geometry>
+    <material name="silver"/>
+  </visual>
+  <collision>
+    <origin xyz="0.01025 0.044348 -0.0853" rpy="0 0 0"/>
+    <geometry>
+      <mesh filename="file://$(find leremix_description)/meshes/arm_base_rotation_servo_1.stl" scale="0.001 0.001 0.001"/>
+    </geometry>
+  </collision>
+</link>
+<link name="arm_base_rotation_link_1">
+  <inertial>
+    <origin xyz="-0.0002718182200486687 -0.03155587105255636 -0.00954044964992927" rpy="0 0 0"/>
+    <mass value="0.5385469320676795"/>
+    <inertia ixx="0.000375" iyy="0.000341" izz="0.000154" ixy="1e-06" iyz="3.6e-05" ixz="3e-06"/>
+  </inertial>
+  <visual>
+    <origin xyz="0.0 0.077148 -0.1199" rpy="0 0 0"/>
+    <geometry>
+      <mesh filename="file://$(find leremix_description)/meshes/arm_base_rotation_link_1.stl" scale="0.001 0.001 0.001"/>
+    </geometry>
+    <material name="silver"/>
+  </visual>
+  <collision>
+    <origin xyz="0.0 0.077148 -0.1199" rpy="0 0 0"/>
+    <geometry>
+      <mesh filename="file://$(find leremix_description)/meshes/arm_base_rotation_link_1.stl" scale="0.001 0.001 0.001"/>
+    </geometry>
+  </collision>
+</link>
+<link name="arm_base_rotation_link_cover_1">
+  <inertial>
+    <origin xyz="0.02324954458129752 0.00949422660202355 -0.0026582098379117625" rpy="0 0 0"/>
+    <mass value="0.10853073755546007"/>
+    <inertia ixx="2.7e-05" iyy="4.6e-05" izz="5.8e-05" ixy="0.0" iyz="0.0" ixz="-0.0"/>
+  </inertial>
+  <visual>
+    <origin xyz="0.023 0.117998 -0.1431" rpy="0 0 0"/>
+    <geometry>
+      <mesh filename="file://$(find leremix_description)/meshes/arm_base_rotation_link_cover_1.stl" scale="0.001 0.001 0.001"/>
+    </geometry>
+    <material name="silver"/>
+  </visual>
+  <collision>
+    <origin xyz="0.023 0.117998 -0.1431" rpy="0 0 0"/>
+    <geometry>
+      <mesh filename="file://$(find leremix_description)/meshes/arm_base_rotation_link_cover_1.stl" scale="0.001 0.001 0.001"/>
+    </geometry>
+  </collision>
+</link>
+<link name="arm_shoulder_servo_1">
+  <inertial>
+    <origin xyz="-0.016027313578788078 0.010249995380535046 0.019999027563219196" rpy="0 0 0"/>
+    <mass value="0.2843033831904074"/>
+    <inertia ixx="6.2e-05" iyy="7.3e-05" izz="4e-05" ixy="-0.0" iyz="0.0" ixz="1e-06"/>
+  </inertial>
+  <visual>
+    <origin xyz="-0.0163 0.117998 -0.1393" rpy="0 0 0"/>
+    <geometry>
+      <mesh filename="file://$(find leremix_description)/meshes/arm_shoulder_servo_1.stl" scale="0.001 0.001 0.001"/>
+    </geometry>
+    <material name="silver"/>
+  </visual>
+  <collision>
+    <origin xyz="-0.0163 0.117998 -0.1393" rpy="0 0 0"/>
+    <geometry>
+      <mesh filename="file://$(find leremix_description)/meshes/arm_shoulder_servo_1.stl" scale="0.001 0.001 0.001"/>
     </geometry>
   </collision>
@@ -44,19 +104,19 @@
 <link name="arm_shoulder_link_1">
   <inertial>
-    <origin xyz="-0.05439041310030922 0.019699384606440277 -0.020185957481023337" rpy="0 0 0"/>
+    <origin xyz="0.019699275433964603 0.055943201517018516 -0.015368254886744204" rpy="0 0 0"/>
     <mass value="0.9906249126045027"/>
-    <inertia ixx="0.000624" iyy="0.001251" izz="0.001489" ixy="-7e-06" iyz="-3e-06" ixz="-0.000385"/>
-  </inertial>
-  <visual>
-    <origin xyz="-0.107007 0.01817 -0.169539" rpy="0 0 0"/>
-    <geometry>
-      <mesh filename="file://$(find LeRemix_description)/meshes/arm_shoulder_link_1.stl" scale="0.001 0.001 0.001"/>
-    </geometry>
-    <material name="silver"/>
-  </visual>
-  <collision>
-    <origin xyz="-0.107007 0.01817 -0.169539" rpy="0 0 0"/>
-    <geometry>
-      <mesh filename="file://$(find LeRemix_description)/meshes/arm_shoulder_link_1.stl" scale="0.001 0.001 0.001"/>
+    <inertia ixx="0.001251" iyy="0.000563" izz="0.001549" ixy="8e-06" iyz="0.000304" ixz="-3e-06"/>
+  </inertial>
+  <visual>
+    <origin xyz="0.0183 0.107748 -0.1721" rpy="0 0 0"/>
+    <geometry>
+      <mesh filename="file://$(find leremix_description)/meshes/arm_shoulder_link_1.stl" scale="0.001 0.001 0.001"/>
+    </geometry>
+    <material name="silver"/>
+  </visual>
+  <collision>
+    <origin xyz="0.0183 0.107748 -0.1721" rpy="0 0 0"/>
+    <geometry>
+      <mesh filename="file://$(find leremix_description)/meshes/arm_shoulder_link_1.stl" scale="0.001 0.001 0.001"/>
     </geometry>
   </collision>
@@ -64,19 +124,19 @@
 <link name="arm_elbow_servo_1">
   <inertial>
-    <origin xyz="-0.016472070877660654 -0.016027204406308133 0.015286802190772275" rpy="0 0 0"/>
+    <origin xyz="-0.016027313578784258 0.015077042423429984 0.016664878981845155" rpy="0 0 0"/>
     <mass value="0.2843033831904074"/>
-    <inertia ixx="7e-05" iyy="6.2e-05" izz="4.4e-05" ixy="-0.0" iyz="1e-06" ixz="1.1e-05"/>
-  </inertial>
-  <visual>
-    <origin xyz="-0.0125 -0.01793 -0.130033" rpy="0 0 0"/>
-    <geometry>
-      <mesh filename="file://$(find LeRemix_description)/meshes/arm_elbow_servo_1.stl" scale="0.001 0.001 0.001"/>
-    </geometry>
-    <material name="silver"/>
-  </visual>
-  <collision>
-    <origin xyz="-0.0125 -0.01793 -0.130033" rpy="0 0 0"/>
-    <geometry>
-      <mesh filename="file://$(find LeRemix_description)/meshes/arm_elbow_servo_1.stl" scale="0.001 0.001 0.001"/>
+    <inertia ixx="6.2e-05" iyy="7.1e-05" izz="4.2e-05" ixy="0.0" iyz="-8e-06" ixz="1e-06"/>
+  </inertial>
+  <visual>
+    <origin xyz="-0.0178 0.010157 -0.140981" rpy="0 0 0"/>
+    <geometry>
+      <mesh filename="file://$(find leremix_description)/meshes/arm_elbow_servo_1.stl" scale="0.001 0.001 0.001"/>
+    </geometry>
+    <material name="silver"/>
+  </visual>
+  <collision>
+    <origin xyz="-0.0178 0.010157 -0.140981" rpy="0 0 0"/>
+    <geometry>
+      <mesh filename="file://$(find leremix_description)/meshes/arm_elbow_servo_1.stl" scale="0.001 0.001 0.001"/>
     </geometry>
   </collision>
@@ -84,19 +144,19 @@
 <link name="arm_elbow_link_1">
   <inertial>
-    <origin xyz="0.05832603889171534 0.015214739326452977 0.021377048894272332" rpy="0 0 0"/>
+    <origin xyz="0.015214630153977244 -0.05832612231118732 0.021376936225360188" rpy="0 0 0"/>
     <mass value="0.8772447501056027"/>
-    <inertia ixx="0.000473" iyy="0.000993" izz="0.001135" ixy="-0.000109" iyz="-4.1e-05" ixz="-0.000289"/>
-  </inertial>
-  <visual>
-    <origin xyz="0.00835 0.01667 -0.157349" rpy="0 0 0"/>
-    <geometry>
-      <mesh filename="file://$(find LeRemix_description)/meshes/arm_elbow_link_1.stl" scale="0.001 0.001 0.001"/>
-    </geometry>
-    <material name="silver"/>
-  </visual>
-  <collision>
-    <origin xyz="0.00835 0.01667 -0.157349" rpy="0 0 0"/>
-    <geometry>
-      <mesh filename="file://$(find LeRemix_description)/meshes/arm_elbow_link_1.stl" scale="0.001 0.001 0.001"/>
+    <inertia ixx="0.000993" iyy="0.000473" izz="0.001135" ixy="0.000109" iyz="0.000289" ixz="-4.1e-05"/>
+  </inertial>
+  <visual>
+    <origin xyz="0.0168 -0.008233 -0.170011" rpy="0 0 0"/>
+    <geometry>
+      <mesh filename="file://$(find leremix_description)/meshes/arm_elbow_link_1.stl" scale="0.001 0.001 0.001"/>
+    </geometry>
+    <material name="silver"/>
+  </visual>
+  <collision>
+    <origin xyz="0.0168 -0.008233 -0.170011" rpy="0 0 0"/>
+    <geometry>
+      <mesh filename="file://$(find leremix_description)/meshes/arm_elbow_link_1.stl" scale="0.001 0.001 0.001"/>
     </geometry>
   </collision>
@@ -104,19 +164,19 @@
 <link name="arm_wrist_tilt_servo_1">
   <inertial>
-    <origin xyz="0.02197013497411679 -0.016027204406307824 -0.004724364582700924" rpy="0 0 0"/>
+    <origin xyz="-0.016027313578783595 -0.021970218393585247 -0.004724477251611736" rpy="0 0 0"/>
     <mass value="0.2843033831904074"/>
-    <inertia ixx="4.2e-05" iyy="6.2e-05" izz="7.1e-05" ixy="1e-06" iyz="0.0" ixz="-8e-06"/>
-  </inertial>
-  <visual>
-    <origin xyz="-0.083248 -0.01943 -0.207129" rpy="0 0 0"/>
-    <geometry>
-      <mesh filename="file://$(find LeRemix_description)/meshes/arm_wrist_tilt_servo_1.stl" scale="0.001 0.001 0.001"/>
-    </geometry>
-    <material name="silver"/>
-  </visual>
-  <collision>
-    <origin xyz="-0.083248 -0.01943 -0.207129" rpy="0 0 0"/>
-    <geometry>
-      <mesh filename="file://$(find LeRemix_description)/meshes/arm_wrist_tilt_servo_1.stl" scale="0.001 0.001 0.001"/>
+    <inertia ixx="6.2e-05" iyy="4.2e-05" izz="7.1e-05" ixy="-1e-06" iyz="8e-06" ixz="0.0"/>
+  </inertial>
+  <visual>
+    <origin xyz="-0.0193 0.083365 -0.219791" rpy="0 0 0"/>
+    <geometry>
+      <mesh filename="file://$(find leremix_description)/meshes/arm_wrist_tilt_servo_1.stl" scale="0.001 0.001 0.001"/>
+    </geometry>
+    <material name="silver"/>
+  </visual>
+  <collision>
+    <origin xyz="-0.0193 0.083365 -0.219791" rpy="0 0 0"/>
+    <geometry>
+      <mesh filename="file://$(find leremix_description)/meshes/arm_wrist_tilt_servo_1.stl" scale="0.001 0.001 0.001"/>
     </geometry>
   </collision>
@@ -124,19 +184,19 @@
 <link name="arm_wrist_link_1">
   <inertial>
-    <origin xyz="0.02004856305995592 0.01680964179048719 -0.017145371524283942" rpy="0 0 0"/>
+    <origin xyz="0.016809532618010315 -0.025935209469899856 -0.0048241515605357554" rpy="0 0 0"/>
     <mass value="0.2392168278135931"/>
-    <inertia ixx="0.000157" iyy="0.000115" izz="0.000169" ixy="5e-06" iyz="-4e-06" ixz="3.6e-05"/>
-  </inertial>
-  <visual>
-    <origin xyz="-0.117583 0.01517 -0.205718" rpy="0 0 0"/>
-    <geometry>
-      <mesh filename="file://$(find LeRemix_description)/meshes/arm_wrist_link_1.stl" scale="0.001 0.001 0.001"/>
-    </geometry>
-    <material name="silver"/>
-  </visual>
-  <collision>
-    <origin xyz="-0.117583 0.01517 -0.205718" rpy="0 0 0"/>
-    <geometry>
-      <mesh filename="file://$(find LeRemix_description)/meshes/arm_wrist_link_1.stl" scale="0.001 0.001 0.001"/>
+    <inertia ixx="0.000115" iyy="0.000129" izz="0.000197" ixy="-7e-06" iyz="-1.3e-05" ixz="-1e-06"/>
+  </inertial>
+  <visual>
+    <origin xyz="0.0153 0.1177 -0.21838" rpy="0 0 0"/>
+    <geometry>
+      <mesh filename="file://$(find leremix_description)/meshes/arm_wrist_link_1.stl" scale="0.001 0.001 0.001"/>
+    </geometry>
+    <material name="silver"/>
+  </visual>
+  <collision>
+    <origin xyz="0.0153 0.1177 -0.21838" rpy="0 0 0"/>
+    <geometry>
+      <mesh filename="file://$(find leremix_description)/meshes/arm_wrist_link_1.stl" scale="0.001 0.001 0.001"/>
     </geometry>
   </collision>
@@ -144,19 +204,19 @@
 <link name="arm_wrist_roll_servo_1">
   <inertial>
-    <origin xyz="-0.018454007185755128 0.01599816538563275 0.002254236765901807" rpy="0 0 0"/>
+    <origin xyz="0.015998056213156815 0.017108254314661786 -0.00727437724496513" rpy="0 0 0"/>
     <mass value="0.2799142523131049"/>
-    <inertia ixx="6.5e-05" iyy="3.8e-05" izz="6.7e-05" ixy="-1e-06" iyz="1e-06" ixz="5e-06"/>
-  </inertial>
-  <visual>
-    <origin xyz="-0.168611 0.02407 -0.175716" rpy="0 0 0"/>
-    <geometry>
-      <mesh filename="file://$(find LeRemix_description)/meshes/arm_wrist_roll_servo_1.stl" scale="0.001 0.001 0.001"/>
-    </geometry>
-    <material name="silver"/>
-  </visual>
-  <collision>
-    <origin xyz="-0.168611 0.02407 -0.175716" rpy="0 0 0"/>
-    <geometry>
-      <mesh filename="file://$(find LeRemix_description)/meshes/arm_wrist_roll_servo_1.stl" scale="0.001 0.001 0.001"/>
+    <inertia ixx="3.8e-05" iyy="6.1e-05" izz="7.1e-05" ixy="1e-06" iyz="-2e-06" ixz="0.0"/>
+  </inertial>
+  <visual>
+    <origin xyz="0.0242 0.176892 -0.217911" rpy="0 0 0"/>
+    <geometry>
+      <mesh filename="file://$(find leremix_description)/meshes/arm_wrist_roll_servo_1.stl" scale="0.001 0.001 0.001"/>
+    </geometry>
+    <material name="silver"/>
+  </visual>
+  <collision>
+    <origin xyz="0.0242 0.176892 -0.217911" rpy="0 0 0"/>
+    <geometry>
+      <mesh filename="file://$(find leremix_description)/meshes/arm_wrist_roll_servo_1.stl" scale="0.001 0.001 0.001"/>
     </geometry>
   </collision>
@@ -164,19 +224,19 @@
 <link name="arm_gripper_1">
   <inertial>
-    <origin xyz="0.01931093722742444 0.012976580613095201 -0.02252356144231421" rpy="0 0 0"/>
+    <origin xyz="0.012976471440619062 -0.027985575300278148 -0.009850406095537195" rpy="0 0 0"/>
     <mass value="0.44698022927880193"/>
-    <inertia ixx="0.000255" iyy="0.000308" izz="0.000237" ixy="-3e-05" iyz="4.4e-05" ixz="8.2e-05"/>
-  </inertial>
-  <visual>
-    <origin xyz="-0.164095 -0.00493 -0.166097" rpy="0 0 0"/>
-    <geometry>
-      <mesh filename="file://$(find LeRemix_description)/meshes/arm_gripper_1.stl" scale="0.001 0.001 0.001"/>
-    </geometry>
-    <material name="silver"/>
-  </visual>
-  <collision>
-    <origin xyz="-0.164095 -0.00493 -0.166097" rpy="0 0 0"/>
-    <geometry>
-      <mesh filename="file://$(find LeRemix_description)/meshes/arm_gripper_1.stl" scale="0.001 0.001 0.001"/>
+    <inertia ixx="0.000308" iyy="0.000179" izz="0.000313" ixy="4.8e-05" iyz="-4.9e-05" ixz="2.3e-05"/>
+  </inertial>
+  <visual>
+    <origin xyz="-0.0048 0.177791 -0.207323" rpy="0 0 0"/>
+    <geometry>
+      <mesh filename="file://$(find leremix_description)/meshes/arm_gripper_1.stl" scale="0.001 0.001 0.001"/>
+    </geometry>
+    <material name="silver"/>
+  </visual>
+  <collision>
+    <origin xyz="-0.0048 0.177791 -0.207323" rpy="0 0 0"/>
+    <geometry>
+      <mesh filename="file://$(find leremix_description)/meshes/arm_gripper_1.stl" scale="0.001 0.001 0.001"/>
     </geometry>
   </collision>
@@ -184,19 +244,19 @@
 <link name="arm_gripper_servo_1">
   <inertial>
-    <origin xyz="0.02230864527990775 -0.012507702080551863 0.010382401144092585" rpy="0 0 0"/>
+    <origin xyz="-0.012507811253028377 -0.014128197579570095 0.020144958135724172" rpy="0 0 0"/>
     <mass value="0.2843033831904074"/>
-    <inertia ixx="6.7e-05" iyy="4.3e-05" izz="6.5e-05" ixy="5e-06" iyz="6e-06" ixz="-8e-06"/>
-  </inertial>
-  <visual>
-    <origin xyz="-0.161113 -0.010962 -0.142741" rpy="0 0 0"/>
-    <geometry>
-      <mesh filename="file://$(find LeRemix_description)/meshes/arm_gripper_servo_1.stl" scale="0.001 0.001 0.001"/>
-    </geometry>
-    <material name="silver"/>
-  </visual>
-  <collision>
-    <origin xyz="-0.161113 -0.010962 -0.142741" rpy="0 0 0"/>
-    <geometry>
-      <mesh filename="file://$(find LeRemix_description)/meshes/arm_gripper_servo_1.stl" scale="0.001 0.001 0.001"/>
+    <inertia ixx="4.3e-05" iyy="7.3e-05" izz="5.9e-05" ixy="-1e-06" iyz="3e-06" ixz="8e-06"/>
+  </inertial>
+  <visual>
+    <origin xyz="-0.010832 0.186887 -0.185606" rpy="0 0 0"/>
+    <geometry>
+      <mesh filename="file://$(find leremix_description)/meshes/arm_gripper_servo_1.stl" scale="0.001 0.001 0.001"/>
+    </geometry>
+    <material name="silver"/>
+  </visual>
+  <collision>
+    <origin xyz="-0.010832 0.186887 -0.185606" rpy="0 0 0"/>
+    <geometry>
+      <mesh filename="file://$(find leremix_description)/meshes/arm_gripper_servo_1.stl" scale="0.001 0.001 0.001"/>
     </geometry>
   </collision>
@@ -204,259 +264,259 @@
 <link name="arm_jaw_1">
   <inertial>
-    <origin xyz="0.009963247508557482 -0.005399256834318277 -0.0350732340426807" rpy="0 0 0"/>
+    <origin xyz="-0.005398366006794445 -0.026165090582212835 -0.0253929839303193" rpy="0 0 0"/>
     <mass value="0.1586808414280307"/>
-    <inertia ixx="4.5e-05" iyy="8.4e-05" izz="5.1e-05" ixy="-9e-06" iyz="-0.0" ixz="2.4e-05"/>
-  </inertial>
-  <visual>
-    <origin xyz="-0.197702 0.006426 -0.169888" rpy="0 0 0"/>
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