Commit message: finally fixed urdf joints

File: ros/src/leremix_gazebo/urdf/gazebo_configs.xacro (robot description, xacro)
@@ -17,5 +17,4 @@
   <self_collide>true</self_collide>
   <gravity>true</gravity>
-  <material>Gazebo/DarkGrey</material>
 </gazebo>
 <gazebo reference="arm_base_rotation_servo_1">
@@ -23,5 +22,19 @@
   <mu2>0.2</mu2>
   <self_collide>true</self_collide>
-  <material>Gazebo/Grey</material>
+</gazebo>
+<gazebo reference="arm_base_rotation_link_1">
+  <mu1>0.2</mu1>
+  <mu2>0.2</mu2>
+  <self_collide>true</self_collide>
+</gazebo>
+<gazebo reference="arm_base_rotation_link_cover_1">
+  <mu1>0.2</mu1>
+  <mu2>0.2</mu2>
+  <self_collide>true</self_collide>
+</gazebo>
+<gazebo reference="arm_shoulder_servo_1">
+  <mu1>0.2</mu1>
+  <mu2>0.2</mu2>
+  <self_collide>true</self_collide>
 </gazebo>
 <gazebo reference="arm_shoulder_link_1">
@@ -29,5 +42,4 @@
   <mu2>0.2</mu2>
   <self_collide>true</self_collide>
-  <material>Gazebo/DarkGrey</material>
 </gazebo>
 <gazebo reference="arm_elbow_servo_1">
@@ -35,5 +47,4 @@
   <mu2>0.2</mu2>
   <self_collide>true</self_collide>
-  <material>Gazebo/Grey</material>
 </gazebo>
 <gazebo reference="arm_elbow_link_1">
@@ -41,5 +52,4 @@
   <mu2>0.2</mu2>
   <self_collide>true</self_collide>
-  <material>Gazebo/DarkGrey</material>
 </gazebo>
 <gazebo reference="arm_wrist_tilt_servo_1">
@@ -47,5 +57,4 @@
   <mu2>0.2</mu2>
   <self_collide>true</self_collide>
-  <material>Gazebo/Grey</material>
 </gazebo>
 <gazebo reference="arm_wrist_link_1">
@@ -53,5 +62,4 @@
   <mu2>0.2</mu2>
   <self_collide>true</self_collide>
-  <material>Gazebo/DarkGrey</material>
 </gazebo>
 <gazebo reference="arm_wrist_roll_servo_1">
@@ -59,5 +67,4 @@
   <mu2>0.2</mu2>
   <self_collide>true</self_collide>
-  <material>Gazebo/Grey</material>
 </gazebo>
 <gazebo reference="arm_gripper_1">
@@ -65,5 +72,4 @@
   <mu2>0.2</mu2>
   <self_collide>true</self_collide>
-  <material>Gazebo/DarkGrey</material>
 </gazebo>
 <gazebo reference="arm_gripper_servo_1">
@@ -71,5 +77,4 @@
   <mu2>0.2</mu2>
   <self_collide>true</self_collide>
-  <material>Gazebo/Grey</material>
 </gazebo>
 <gazebo reference="arm_jaw_1">
@@ -77,5 +82,4 @@
   <mu2>0.2</mu2>
   <self_collide>true</self_collide>
-  <material>Gazebo/DarkGrey</material>
 </gazebo>
 <gazebo reference="right_servo_mount_1">
@@ -83,5 +87,4 @@
   <mu2>0.2</mu2>
   <self_collide>true</self_collide>
-  <material>Gazebo/DarkGrey</material>
 </gazebo>
 <gazebo reference="right_servo_1">
@@ -89,11 +92,4 @@
   <mu2>0.2</mu2>
   <self_collide>true</self_collide>
-  <material>Gazebo/Grey</material>
-</gazebo>
-<gazebo reference="right_wheel_mount_1">
-  <mu1>0.2</mu1>
-  <mu2>0.2</mu2>
-  <self_collide>true</self_collide>
-  <material>Gazebo/DarkGrey</material>
 </gazebo>
 <gazebo reference="back_servo_mount_1">
@@ -101,5 +97,4 @@
   <mu2>0.2</mu2>
   <self_collide>true</self_collide>
-  <material>Gazebo/DarkGrey</material>
 </gazebo>
 <gazebo reference="left_servo_mount_1">
@@ -107,5 +102,4 @@
   <mu2>0.2</mu2>
   <self_collide>true</self_collide>
-  <material>Gazebo/DarkGrey</material>
 </gazebo>
 <gazebo reference="back_servo_1">
@@ -113,5 +107,4 @@
   <mu2>0.2</mu2>
   <self_collide>true</self_collide>
-  <material>Gazebo/Grey</material>
 </gazebo>
 <gazebo reference="back_wheel_mount_1">
@@ -119,5 +112,144 @@
   <mu2>0.2</mu2>
   <self_collide>true</self_collide>
-  <material>Gazebo/DarkGrey</material>
+</gazebo>
+<gazebo reference="back_wheel_1">
+  <mu1>0.2</mu1>
+  <mu2>0.2</mu2>
+  <self_collide>true</self_collide>
+</gazebo>
+<gazebo reference="left_servo_1">
+  <mu1>0.2</mu1>
+  <mu2>0.2</mu2>
+  <self_collide>true</self_collide>
+</gazebo>
+<gazebo reference="left_wheel_mount_1">
+  <mu1>0.2</mu1>
+  <mu2>0.2</mu2>
+  <self_collide>true</self_collide>
+</gazebo>
+<gazebo reference="orin_1">
+  <mu1>0.2</mu1>
+  <mu2>0.2</mu2>
+  <self_collide>true</self_collide>
+</gazebo>
+<gazebo reference="orin_mount_1">
+  <mu1>0.2</mu1>
+  <mu2>0.2</mu2>
+  <self_collide>true</self_collide>
+</gazebo>
+<gazebo reference="battery_stopper_1">
+  <mu1>0.2</mu1>
+  <mu2>0.2</mu2>
+  <self_collide>true</self_collide>
+</gazebo>
+<gazebo reference="usb_pd_mount_1">
+  <mu1>0.2</mu1>
+  <mu2>0.2</mu2>
+  <self_collide>true</self_collide>
+</gazebo>
+<gazebo reference="arm_base_1">
+  <mu1>0.2</mu1>
+  <mu2>0.2</mu2>
+  <self_collide>true</self_collide>
+</gazebo>
+<gazebo reference="imu_1">
+  <mu1>0.2</mu1>
+  <mu2>0.2</mu2>
+  <self_collide>true</self_collide>
+</gazebo>
+<gazebo reference="imu_mount_1">
+  <mu1>0.2</mu1>
+  <mu2>0.2</mu2>
+  <self_collide>true</self_collide>
+</gazebo>
+<gazebo reference="hex_1__1__1">
+  <mu1>0.2</mu1>
+  <mu2>0.2</mu2>
+  <self_collide>true</self_collide>
+</gazebo>
+<gazebo reference="just_the_tower_v1_1">
+  <mu1>0.2</mu1>
+  <mu2>0.2</mu2>
+  <self_collide>true</self_collide>
+</gazebo>
+<gazebo reference="support_v1_1">
+  <mu1>0.2</mu1>
+  <mu2>0.2</mu2>
+  <self_collide>true</self_collide>
+</gazebo>
+<gazebo reference="head_camera_1">
+  <mu1>0.2</mu1>
+  <mu2>0.2</mu2>
+  <self_collide>true</self_collide>
+</gazebo>
+<gazebo reference="hex_1_1">
+  <mu1>0.2</mu1>
+  <mu2>0.2</mu2>
+  <self_collide>true</self_collide>
+</gazebo>
+<gazebo reference="hex_2_1">
+  <mu1>0.2</mu1>
+  <mu2>0.2</mu2>
+  <self_collide>true</self_collide>
+</gazebo>
+<gazebo reference="hex_1__1___1__1">
+  <mu1>0.2</mu1>
+  <mu2>0.2</mu2>
+  <self_collide>true</self_collide>
+</gazebo>
+<gazebo reference="last_floor_v1_1">
+  <mu1>0.2</mu1>
+  <mu2>0.2</mu2>
+  <self_collide>true</self_collide>
+</gazebo>
+<gazebo reference="front_cam_support_1">
+  <mu1>0.2</mu1>
+  <mu2>0.2</mu2>
+  <self_collide>true</self_collide>
+</gazebo>
+<gazebo reference="front_camera_1">
+  <mu1>0.2</mu1>
+  <mu2>0.2</mu2>
+  <self_collide>true</self_collide>
+</gazebo>
+<gazebo reference="hex_3_1">
+  <mu1>0.2</mu1>
+  <mu2>0.2</mu2>
+  <self_collide>true</self_collide>
+</gazebo>
+<gazebo reference="hex_4_1">
+  <mu1>0.2</mu1>
+  <mu2>0.2</mu2>
+  <self_collide>true</self_collide>
+</gazebo>
+<gazebo reference="upper_floor_1">
+  <mu1>0.2</mu1>
+  <mu2>0.2</mu2>
+  <self_collide>true</self_collide>
+</gazebo>
+<gazebo reference="pan_link_1">
+  <mu1>0.2</mu1>
+  <mu2>0.2</mu2>
+  <self_collide>true</self_collide>
+</gazebo>
+<gazebo reference="tilt_servo_1">
+  <mu1>0.2</mu1>
+  <mu2>0.2</mu2>
+  <self_collide>true</self_collide>
+</gazebo>
+<gazebo reference="tilt_link_cover_1">
+  <mu1>0.2</mu1>
+  <mu2>0.2</mu2>
+  <self_collide>true</self_collide>
+</gazebo>
+<gazebo reference="realsense_support_v1_1">
+  <mu1>0.2</mu1>
+  <mu2>0.2</mu2>
+  <self_collide>true</self_collide>
+</gazebo>
+<gazebo reference="pan_servo__1__1">
+  <mu1>0.2</mu1>
+  <mu2>0.2</mu2>
+  <self_collide>true</self_collide>
 </gazebo>
 <gazebo reference="right_wheel_1">
@@ -148,165 +280,3 @@
   <kd>3.5</kd>
 </gazebo>
-<gazebo reference="left_servo_1">
-  <mu1>0.2</mu1>
-  <mu2>0.2</mu2>
-  <self_collide>true</self_collide>
-  <material>Gazebo/Grey</material>
-</gazebo>
-<gazebo reference="left_wheel_mount_1">
-  <mu1>0.2</mu1>
-  <mu2>0.2</mu2>
-  <self_collide>true</self_collide>
-  <material>Gazebo/DarkGrey</material>
-</gazebo>
-<gazebo reference="orin_1">
-  <mu1>0.2</mu1>
-  <mu2>0.2</mu2>
-  <self_collide>true</self_collide>
-  <material>Gazebo/Grey</material>
-</gazebo>
-<gazebo reference="hex_2_1">
-  <mu1>0.2</mu1>
-  <mu2>0.2</mu2>
-  <self_collide>true</self_collide>
-  <material>Gazebo/DarkYellow</material>
-</gazebo>
-<gazebo reference="hex_1_1">
-  <mu1>0.2</mu1>
-  <mu2>0.2</mu2>
-  <self_collide>true</self_collide>
-  <material>Gazebo/DarkYellow</material>
-</gazebo>
-<gazebo reference="hex_3_1">
-  <mu1>0.2</mu1>
-  <mu2>0.2</mu2>
-  <self_collide>true</self_collide>
-  <material>Gazebo/DarkYellow</material>
-</gazebo>
-<gazebo reference="usb_pd_mount_1">
-  <mu1>0.2</mu1>
-  <mu2>0.2</mu2>
-  <self_collide>true</self_collide>
-  <material>Gazebo/DarkGrey</material>
-</gazebo>
-<gazebo reference="imu_1">
-  <mu1>0.2</mu1>
-  <mu2>0.2</mu2>
-  <self_collide>true</self_collide>
-  <material>Gazebo/Grey</material>
-</gazebo>
-<gazebo reference="panny_v1_1">
-  <mu1>0.2</mu1>
-  <mu2>0.2</mu2>
-  <self_collide>true</self_collide>
-  <material>Gazebo/DarkGrey</material>
-</gazebo>
-<gazebo reference="pan_servo_1">
-  <mu1>0.2</mu1>
-  <mu2>0.2</mu2>
-  <self_collide>true</self_collide>
-  <material>Gazebo/Grey</material>
-</gazebo>
-<gazebo reference="camera_tilt_mount_v1_1">
-  <mu1>0.2</mu1>
-  <mu2>0.2</mu2>
-  <self_collide>true</self_collide>
-  <material>Gazebo/DarkGrey</material>
-</gazebo>
-<gazebo reference="camera_1">
-  <mu1>0.2</mu1>
-  <mu2>0.2</mu2>
-  <self_collide>true</self_collide>
-    <material>Gazebo/Grey</material>
-</gazebo>
-<gazebo reference="right_baseus_mount_v1_1">
-  <mu1>0.2</mu1>
-  <mu2>0.2</mu2>
-  <self_collide>true</self_collide>
-    <material>Gazebo/DarkGrey</material>
-</gazebo>
-<gazebo reference="arm_shoulder_servo_1">
-  <mu1>0.2</mu1>
-  <mu2>0.2</mu2>
-  <self_collide>true</self_collide>
-  <material>Gazebo/Grey</material>
-</gazebo>
-<gazebo reference="arm_base_rotation_link_cover_1">
-  <mu1>0.2</mu1>
-  <mu2>0.2</mu2>
-  <self_collide>true</self_collide>
-  <material>Gazebo/DarkGrey</material>
-</gazebo>
-<gazebo reference="orin_mount_1">
-  <mu1>0.2</mu1>
-  <mu2>0.2</mu2>
-  <self_collide>true</self_collide>
-  <material>Gazebo/DarkGrey</material>
-</gazebo>
-<gazebo reference="arm_base_1">
-  <mu1>0.2</mu1>
-  <mu2>0.2</mu2>
-  <self_collide>true</self_collide>
-  <material>Gazebo/DarkGrey</material>
-</gazebo>
-<gazebo reference="imu_mount_1">
-  <mu1>0.2</mu1>
-  <mu2>0.2</mu2>
-  <self_collide>true</self_collide>
-  <material>Gazebo/DarkGrey</material>
-</gazebo>
-<gazebo reference="hex_5_1">
-  <mu1>0.2</mu1>
-  <mu2>0.2</mu2>
-  <self_collide>true</self_collide>
-  <material>Gazebo/DarkYellow</material>
-</gazebo>
-<gazebo reference="last_floor_v1_1">
-  <mu1>0.2</mu1>
-  <mu2>0.2</mu2>
-  <self_collide>true</self_collide>
-  <material>Gazebo/DarkGrey</material>
-</gazebo>
-<gazebo reference="left_baseus_mount_v1_1">
-  <mu1>0.2</mu1>
-  <mu2>0.2</mu2>
-  <self_collide>true</self_collide>
-  <material>Gazebo/DarkGrey</material>
-</gazebo>
-<gazebo reference="baseus_pack_v1_1">
-  <mu1>0.2</mu1>
-  <mu2>0.2</mu2>
-  <self_collide>true</self_collide>
-  <material>Gazebo/Silver</material>
-</gazebo>
-<gazebo reference="hex_7_1">
-  <mu1>0.2</mu1>
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
File: ros/src/leremix_gazebo/urdf/gazebo_interfaces.xacro (robot description, xacro)
@@ -5,5 +5,5 @@
             <plugin>gazebo_ros2_control/GazeboSystem</plugin>
         </hardware>
-        <joint name="back_motor_rotation">
+        <joint name="wheel1_rotation">
             <command_interface name="velocity">
                 <param name="min">-10</param>
@@ -13,5 +13,5 @@
             <state_interface name="velocity"/>
         </joint>
-        <joint name="left_motor_rotation">
+        <joint name="wheel2_rotation">
             <command_interface name="velocity">
                 <param name="min">-10</param>
@@ -21,5 +21,5 @@
             <state_interface name="velocity"/>
         </joint>
-        <joint name="right_motor_rotation">
+        <joint name="wheel3_rotation">
             <command_interface name="velocity">
                 <param name="min">-10</param>
@@ -30,4 +30,9 @@
         </joint>
         <joint name="camera_tilt">
+          <command_interface name="position">
+            </command_interface>
+            <state_interface name="position" />
+        </joint>
+        <joint name="camera_pan">
           <command_interface name="position">
             </command_interface>
