Commit message: added lidar and wrist camera urdf

File: ros/src/leremix_description/urdf/LeRemix.xacro (robot description, xacro)
@@ -4,7 +4,7 @@
 <link name="base_link">
   <inertial>
-    <origin xyz="3.340802284881761e-05 0.0062553486303636415 0.0025000000000001423" rpy="0 0 0"/>
-    <mass value="1.5793453539076086"/>
-    <inertia ixx="0.005179" iyy="0.00541" izz="0.010582" ixy="3e-06" iyz="-0.0" ixz="0.0"/>
+    <origin xyz="5.866413998148801e-05 0.0062819967824381704 0.001416599330144379" rpy="0 0 0"/>
+    <mass value="0.8949198281645031"/>
+    <inertia ixx="0.003064" iyy="0.002933" izz="0.005996" ixy="-2e-06" iyz="0.0" ixz="0.0"/>
   </inertial>
   <visual>
@@ -24,10 +24,10 @@
 <link name="arm_base_rotation_servo_1">
   <inertial>
-    <origin xyz="0.010249751352689343 -0.01999903218942549 0.016027064924724457" rpy="0 0 0"/>
+    <origin xyz="0.019999044959765788 0.01025034011227997 0.016027263585011595" rpy="0 0 0"/>
     <mass value="0.2843033831904074"/>
-    <inertia ixx="7.3e-05" iyy="4e-05" izz="6.2e-05" ixy="-0.0" iyz="1e-06" ixz="0.0"/>
-  </inertial>
-  <visual>
-    <origin xyz="0.01025 0.044348 -0.0853" rpy="0 0 0"/>
+    <inertia ixx="4e-05" iyy="7.3e-05" izz="6.2e-05" ixy="0.0" iyz="0.0" ixz="-1e-06"/>
+  </inertial>
+  <visual>
+    <origin xyz="-0.050662 0.004002 -0.083133" rpy="0 0 0"/>
     <geometry>
       <mesh filename="file://$(find leremix_description)/meshes/arm_base_rotation_servo_1.stl" scale="0.001 0.001 0.001"/>
@@ -36,5 +36,5 @@
   </visual>
   <collision>
-    <origin xyz="0.01025 0.044348 -0.0853" rpy="0 0 0"/>
+    <origin xyz="-0.050662 0.004002 -0.083133" rpy="0 0 0"/>
     <geometry>
       <mesh filename="file://$(find leremix_description)/meshes/arm_base_rotation_servo_1.stl" scale="0.001 0.001 0.001"/>
@@ -44,10 +44,10 @@
 <link name="arm_base_rotation_link_1">
   <inertial>
-    <origin xyz="-0.0002718182200486687 -0.03155587105255636 -0.00954044964992927" rpy="0 0 0"/>
+    <origin xyz="0.03155588382289583 -0.00027122946045804366 -0.009540250989642243" rpy="0 0 0"/>
     <mass value="0.5385469320676795"/>
-    <inertia ixx="0.000375" iyy="0.000341" izz="0.000154" ixy="1e-06" iyz="3.6e-05" ixz="3e-06"/>
-  </inertial>
-  <visual>
-    <origin xyz="0.0 0.077148 -0.1199" rpy="0 0 0"/>
+    <inertia ixx="0.000341" iyy="0.000375" izz="0.000154" ixy="-1e-06" iyz="3e-06" ixz="-3.6e-05"/>
+  </inertial>
+  <visual>
+    <origin xyz="-0.083462 -0.006248 -0.117733" rpy="0 0 0"/>
     <geometry>
       <mesh filename="file://$(find leremix_description)/meshes/arm_base_rotation_link_1.stl" scale="0.001 0.001 0.001"/>
@@ -56,5 +56,5 @@
   </visual>
   <collision>
-    <origin xyz="0.0 0.077148 -0.1199" rpy="0 0 0"/>
+    <origin xyz="-0.083462 -0.006248 -0.117733" rpy="0 0 0"/>
     <geometry>
       <mesh filename="file://$(find leremix_description)/meshes/arm_base_rotation_link_1.stl" scale="0.001 0.001 0.001"/>
@@ -64,10 +64,10 @@
 <link name="arm_base_rotation_link_cover_1">
   <inertial>
-    <origin xyz="0.02324954458129752 0.00949422660202355 -0.0026582098379117625" rpy="0 0 0"/>
+    <origin xyz="-0.009494213831683473 0.023250133340888265 -0.002658011177624875" rpy="0 0 0"/>
     <mass value="0.10853073755546007"/>
-    <inertia ixx="2.7e-05" iyy="4.6e-05" izz="5.8e-05" ixy="0.0" iyz="0.0" ixz="-0.0"/>
-  </inertial>
-  <visual>
-    <origin xyz="0.023 0.117998 -0.1431" rpy="0 0 0"/>
+    <inertia ixx="4.6e-05" iyy="2.7e-05" izz="5.8e-05" ixy="-0.0" iyz="-0.0" ixz="-0.0"/>
+  </inertial>
+  <visual>
+    <origin xyz="-0.124312 0.016752 -0.140933" rpy="0 0 0"/>
     <geometry>
       <mesh filename="file://$(find leremix_description)/meshes/arm_base_rotation_link_cover_1.stl" scale="0.001 0.001 0.001"/>
@@ -76,5 +76,5 @@
   </visual>
   <collision>
-    <origin xyz="0.023 0.117998 -0.1431" rpy="0 0 0"/>
+    <origin xyz="-0.124312 0.016752 -0.140933" rpy="0 0 0"/>
     <geometry>
       <mesh filename="file://$(find leremix_description)/meshes/arm_base_rotation_link_cover_1.stl" scale="0.001 0.001 0.001"/>
@@ -84,10 +84,10 @@
 <link name="arm_shoulder_servo_1">
   <inertial>
-    <origin xyz="-0.016027313578788078 0.010249995380535046 0.019999027563219196" rpy="0 0 0"/>
+    <origin xyz="-0.010249982610195635 -0.016026724819197403 0.019999226223505806" rpy="0 0 0"/>
     <mass value="0.2843033831904074"/>
-    <inertia ixx="6.2e-05" iyy="7.3e-05" izz="4e-05" ixy="-0.0" iyz="0.0" ixz="1e-06"/>
-  </inertial>
-  <visual>
-    <origin xyz="-0.0163 0.117998 -0.1393" rpy="0 0 0"/>
+    <inertia ixx="7.3e-05" iyy="6.2e-05" izz="4e-05" ixy="0.0" iyz="1e-06" ixz="-0.0"/>
+  </inertial>
+  <visual>
+    <origin xyz="-0.124312 -0.022548 -0.137133" rpy="0 0 0"/>
     <geometry>
       <mesh filename="file://$(find leremix_description)/meshes/arm_shoulder_servo_1.stl" scale="0.001 0.001 0.001"/>
@@ -96,5 +96,5 @@
   </visual>
   <collision>
-    <origin xyz="-0.0163 0.117998 -0.1393" rpy="0 0 0"/>
+    <origin xyz="-0.124312 -0.022548 -0.137133" rpy="0 0 0"/>
     <geometry>
       <mesh filename="file://$(find leremix_description)/meshes/arm_shoulder_servo_1.stl" scale="0.001 0.001 0.001"/>
@@ -104,10 +104,10 @@
 <link name="arm_shoulder_link_1">
   <inertial>
-    <origin xyz="0.019699275433964603 0.055943201517018516 -0.015368254886744204" rpy="0 0 0"/>
+    <origin xyz="-0.055943188746678085 0.01969986419355535 -0.015368056226457844" rpy="0 0 0"/>
     <mass value="0.9906249126045027"/>
-    <inertia ixx="0.001251" iyy="0.000563" izz="0.001549" ixy="8e-06" iyz="0.000304" ixz="-3e-06"/>
-  </inertial>
-  <visual>
-    <origin xyz="0.0183 0.107748 -0.1721" rpy="0 0 0"/>
+    <inertia ixx="0.000563" iyy="0.001251" izz="0.001549" ixy="-8e-06" iyz="-3e-06" ixz="-0.000304"/>
+  </inertial>
+  <visual>
+    <origin xyz="-0.114062 0.012052 -0.169933" rpy="0 0 0"/>
     <geometry>
       <mesh filename="file://$(find leremix_description)/meshes/arm_shoulder_link_1.stl" scale="0.001 0.001 0.001"/>
@@ -116,5 +116,5 @@
   </visual>
   <collision>
-    <origin xyz="0.0183 0.107748 -0.1721" rpy="0 0 0"/>
+    <origin xyz="-0.114062 0.012052 -0.169933" rpy="0 0 0"/>
     <geometry>
       <mesh filename="file://$(find leremix_description)/meshes/arm_shoulder_link_1.stl" scale="0.001 0.001 0.001"/>
@@ -124,10 +124,10 @@
 <link name="arm_elbow_servo_1">
   <inertial>
-    <origin xyz="-0.016027313578784258 0.015077042423429984 0.016664878981845155" rpy="0 0 0"/>
+    <origin xyz="-0.015077029653089111 -0.016026724819193545 0.016665077642131626" rpy="0 0 0"/>
     <mass value="0.2843033831904074"/>
-    <inertia ixx="6.2e-05" iyy="7.1e-05" izz="4.2e-05" ixy="0.0" iyz="-8e-06" ixz="1e-06"/>
-  </inertial>
-  <visual>
-    <origin xyz="-0.0178 0.010157 -0.140981" rpy="0 0 0"/>
+    <inertia ixx="7.1e-05" iyy="6.2e-05" izz="4.2e-05" ixy="-0.0" iyz="1e-06" ixz="8e-06"/>
+  </inertial>
+  <visual>
+    <origin xyz="-0.016471 -0.024048 -0.138814" rpy="0 0 0"/>
     <geometry>
       <mesh filename="file://$(find leremix_description)/meshes/arm_elbow_servo_1.stl" scale="0.001 0.001 0.001"/>
@@ -136,5 +136,5 @@
   </visual>
   <collision>
-    <origin xyz="-0.0178 0.010157 -0.140981" rpy="0 0 0"/>
+    <origin xyz="-0.016471 -0.024048 -0.138814" rpy="0 0 0"/>
     <geometry>
       <mesh filename="file://$(find leremix_description)/meshes/arm_elbow_servo_1.stl" scale="0.001 0.001 0.001"/>
@@ -144,10 +144,10 @@
 <link name="arm_elbow_link_1">
   <inertial>
-    <origin xyz="0.015214630153977244 -0.05832612231118732 0.021376936225360188" rpy="0 0 0"/>
+    <origin xyz="0.05832613508152747 0.015215218913568064 0.02137713488564641" rpy="0 0 0"/>
     <mass value="0.8772447501056027"/>
-    <inertia ixx="0.000993" iyy="0.000473" izz="0.001135" ixy="0.000109" iyz="0.000289" ixz="-4.1e-05"/>
-  </inertial>
-  <visual>
-    <origin xyz="0.0168 -0.008233 -0.170011" rpy="0 0 0"/>
+    <inertia ixx="0.000473" iyy="0.000993" izz="0.001135" ixy="-0.000109" iyz="-4.1e-05" ixz="-0.000289"/>
+  </inertial>
+  <visual>
+    <origin xyz="0.001919 0.010552 -0.167844" rpy="0 0 0"/>
     <geometry>
       <mesh filename="file://$(find leremix_description)/meshes/arm_elbow_link_1.stl" scale="0.001 0.001 0.001"/>
@@ -156,5 +156,5 @@
   </visual>
   <collision>
-    <origin xyz="0.0168 -0.008233 -0.170011" rpy="0 0 0"/>
+    <origin xyz="0.001919 0.010552 -0.167844" rpy="0 0 0"/>
     <geometry>
       <mesh filename="file://$(find leremix_description)/meshes/arm_elbow_link_1.stl" scale="0.001 0.001 0.001"/>
@@ -164,10 +164,10 @@
 <link name="arm_wrist_tilt_servo_1">
   <inertial>
-    <origin xyz="-0.016027313578783595 -0.021970218393585247 -0.004724477251611736" rpy="0 0 0"/>
+    <origin xyz="0.021970231163924825 -0.016026724819192876 -0.004724278591325293" rpy="0 0 0"/>
     <mass value="0.2843033831904074"/>
-    <inertia ixx="6.2e-05" iyy="4.2e-05" izz="7.1e-05" ixy="-1e-06" iyz="8e-06" ixz="0.0"/>
-  </inertial>
-  <visual>
-    <origin xyz="-0.0193 0.083365 -0.219791" rpy="0 0 0"/>
+    <inertia ixx="4.2e-05" iyy="6.2e-05" izz="7.1e-05" ixy="1e-06" iyz="0.0" ixz="-8e-06"/>
+  </inertial>
+  <visual>
+    <origin xyz="-0.089679 -0.025548 -0.217624" rpy="0 0 0"/>
     <geometry>
       <mesh filename="file://$(find leremix_description)/meshes/arm_wrist_tilt_servo_1.stl" scale="0.001 0.001 0.001"/>
@@ -176,5 +176,5 @@
   </visual>
   <collision>
-    <origin xyz="-0.0193 0.083365 -0.219791" rpy="0 0 0"/>
+    <origin xyz="-0.089679 -0.025548 -0.217624" rpy="0 0 0"/>
     <geometry>
       <mesh filename="file://$(find leremix_description)/meshes/arm_wrist_tilt_servo_1.stl" scale="0.001 0.001 0.001"/>
@@ -184,10 +184,10 @@
 <link name="arm_wrist_link_1">
   <inertial>
-    <origin xyz="0.016809532618010315 -0.025935209469899856 -0.0048241515605357554" rpy="0 0 0"/>
+    <origin xyz="0.012975594362619927 0.016810121377602565 -0.02296834504128556" rpy="0 0 0"/>
     <mass value="0.2392168278135931"/>
-    <inertia ixx="0.000115" iyy="0.000129" izz="0.000197" ixy="-7e-06" iyz="-1.3e-05" ixz="-1e-06"/>
-  </inertial>
-  <visual>
-    <origin xyz="0.0153 0.1177 -0.21838" rpy="0 0 0"/>
+    <inertia ixx="0.000182" iyy="0.000115" izz="0.000144" ixy="3e-06" iyz="-6e-06" ixz="3.2e-05"/>
+  </inertial>
+  <visual>
+    <origin xyz="-0.124014 0.009052 -0.216213" rpy="0 0 0"/>
     <geometry>
       <mesh filename="file://$(find leremix_description)/meshes/arm_wrist_link_1.stl" scale="0.001 0.001 0.001"/>
@@ -196,5 +196,5 @@
   </visual>
   <collision>
-    <origin xyz="0.0153 0.1177 -0.21838" rpy="0 0 0"/>
+    <origin xyz="-0.124014 0.009052 -0.216213" rpy="0 0 0"/>
     <geometry>
       <mesh filename="file://$(find leremix_description)/meshes/arm_wrist_link_1.stl" scale="0.001 0.001 0.001"/>
@@ -204,10 +204,10 @@
 <link name="arm_wrist_roll_servo_1">
   <inertial>
-    <origin xyz="0.015998056213156815 0.017108254314661786 -0.00727437724496513" rpy="0 0 0"/>
+    <origin xyz="-0.01656958325728916 0.015998644972749377 0.008429716426542305" rpy="0 0 0"/>
     <mass value="0.2799142523131049"/>
-    <inertia ixx="3.8e-05" iyy="6.1e-05" izz="7.1e-05" ixy="1e-06" iyz="-2e-06" ixz="0.0"/>
-  </inertial>
-  <visual>
-    <origin xyz="0.0242 0.176892 -0.217911" rpy="0 0 0"/>
+    <inertia ixx="6.9e-05" iyy="3.8e-05" izz="6.3e-05" ixy="-1e-06" iyz="1e-06" ixz="5e-06"/>
+  </inertial>
+  <visual>
+    <origin xyz="-0.161703 0.017952 -0.170568" rpy="0 0 0"/>
     <geometry>
       <mesh filename="file://$(find leremix_description)/meshes/arm_wrist_roll_servo_1.stl" scale="0.001 0.001 0.001"/>
@@ -216,5 +216,5 @@
   </visual>
   <collision>
-    <origin xyz="0.0242 0.176892 -0.217911" rpy="0 0 0"/>
+    <origin xyz="-0.161703 0.017952 -0.170568" rpy="0 0 0"/>
     <geometry>
       <mesh filename="file://$(find leremix_description)/meshes/arm_wrist_roll_servo_1.stl" scale="0.001 0.001 0.001"/>
@@ -224,10 +224,10 @@
 <link name="arm_gripper_1">
   <inertial>
-    <origin xyz="0.012976471440619062 -0.027985575300278148 -0.009850406095537195" rpy="0 0 0"/>
+    <origin xyz="0.013339671966003358 -0.013714806926169776 -0.026125553965198" rpy="0 0 0"/>
     <mass value="0.44698022927880193"/>
-    <inertia ixx="0.000308" iyy="0.000179" izz="0.000313" ixy="4.8e-05" iyz="-4.9e-05" ixz="2.3e-05"/>
-  </inertial>
-  <visual>
-    <origin xyz="-0.0048 0.177791 -0.207323" rpy="0 0 0"/>
+    <inertia ixx="0.000294" iyy="0.000301" izz="0.000205" ixy="3e-05" iyz="-4.7e-05" ixz="7.1e-05"/>
+  </inertial>
+  <visual>
+    <origin xyz="-0.15417 -0.011048 -0.163073" rpy="0 0 0"/>
     <geometry>
       <mesh filename="file://$(find leremix_description)/meshes/arm_gripper_1.stl" scale="0.001 0.001 0.001"/>
@@ -236,5 +236,5 @@
   </visual>
   <collision>
-    <origin xyz="-0.0048 0.177791 -0.207323" rpy="0 0 0"/>
+    <origin xyz="-0.15417 -0.011048 -0.163073" rpy="0 0 0"/>
     <geometry>
       <mesh filename="file://$(find leremix_description)/meshes/arm_gripper_1.stl" scale="0.001 0.001 0.001"/>
@@ -244,10 +244,10 @@
 <link name="arm_gripper_servo_1">
   <inertial>
-    <origin xyz="-0.012507811253028377 -0.014128197579570095 0.020144958135724172" rpy="0 0 0"/>
+    <origin xyz="-0.007975468163954197 0.020789656863227802 -0.01631207348591407" rpy="0 0 0"/>
     <mass value="0.2843033831904074"/>
-    <inertia ixx="4.3e-05" iyy="7.3e-05" izz="5.9e-05" ixy="-1e-06" iyz="3e-06" ixz="8e-06"/>
-  </inertial>
-  <visual>
-    <origin xyz="-0.010832 0.186887 -0.185606" rpy="0 0 0"/>
+    <inertia ixx="6.4e-05" iyy="4e-05" izz="7.1e-05" ixy="-0.0" iyz="-0.0" ixz="-5e-06"/>
+  </inertial>
+  <visual>
+    <origin xyz="-0.173846 0.00275 -0.159436" rpy="0 0 0"/>
     <geometry>
       <mesh filename="file://$(find leremix_description)/meshes/arm_gripper_servo_1.stl" scale="0.001 0.001 0.001"/>
@@ -256,5 +256,5 @@
   </visual>
   <collision>
-    <origin xyz="-0.010832 0.186887 -0.185606" rpy="0 0 0"/>
+    <origin xyz="-0.173846 0.00275 -0.159436" rpy="0 0 0"/>
     <geometry>
       <mesh filename="file://$(find leremix_description)/meshes/arm_gripper_servo_1.stl" scale="0.001 0.001 0.001"/>
@@ -264,10 +264,10 @@
 <link name="arm_jaw_1">
   <inertial>
-    <origin xyz="-0.005398366006794445 -0.026165090582212835 -0.0253929839303193" rpy="0 0 0"/>
+    <origin xyz="0.032905631581261585 -0.003660190112443975 -0.016197173267020665" rpy="0 0 0"/>
     <mass value="0.1586808414280307"/>
-    <inertia ixx="8.4e-05" iyy="2.6e-05" izz="7.1e-05" ixy="7e-06" iyz="-1e-05" ixz="-4e-06"/>
-  </inertial>
-  <visual>
-    <origin xyz="0.006557 0.205 -0.22741" rpy="0 0 0"/>
+    <inertia ixx="6.1e-05" iyy="8.6e-05" izz="3.4e-05" ixy="4e-06" iyz="-5e-06" ixz="1.9e-05"/>
+  </inertial>
+  <visual>
+    <origin xyz="-0.150306 -0.03177 -0.134291" rpy="0 0 0"/>
     <geometry>
       <mesh filename="file://$(find leremix_description)/meshes/arm_jaw_1.stl" scale="0.001 0.001 0.001"/>
@@ -276,5 +276,5 @@
   </visual>
   <collision>
-    <origin xyz="0.006557 0.205 -0.22741" rpy="0 0 0"/>
+    <origin xyz="-0.150306 -0.03177 -0.134291" rpy="0 0 0"/>
     <geometry>
       <mesh filename="file://$(find leremix_description)/meshes/arm_jaw_1.stl" scale="0.001 0.001 0.001"/>
@@ -284,10 +284,10 @@
 <link name="right_servo_mount_1">
   <inertial>
-    <origin xyz="0.005194056332463476 -0.02008773112678317 0.02361159724929678" rpy="0 0 0"/>
+    <origin xyz="0.02008674389712354 0.005193645092054736 0.023611795909587813" rpy="0 0 0"/>
     <mass value="0.14423806644766202"/>
-    <inertia ixx="6.4e-05" iyy="5.5e-05" izz="5.3e-05" ixy="8e-06" iyz="-1e-06" ixz="-1e-06"/>
-  </inertial>
-  <visual>
-    <origin xyz="0.079282 0.022679 -0.005" rpy="0 0 0"/>
+    <inertia ixx="5.5e-05" iyy="6.4e-05" izz="5.3e-05" ixy="-8e-06" iyz="-1e-06" ixz="1e-06"/>
+  </inertial>
+  <visual>
+    <origin xyz="-0.028994 0.073033 -0.002833" rpy="0 0 0"/>
     <geometry>
       <mesh filename="file://$(find leremix_description)/meshes/right_servo_mount_1.stl" scale="0.001 0.001 0.001"/>
@@ -296,5 +296,5 @@
   </visual>
   <collision>
-    <origin xyz="0.079282 0.022679 -0.005" rpy="0 0 0"/>
+    <origin xyz="-0.028994 0.073033 -0.002833" rpy="0 0 0"/>
     <geometry>
       <mesh filename="file://$(find leremix_description)/meshes/right_servo_mount_1.stl" scale="0.001 0.001 0.001"/>
@@ -304,10 +304,10 @@
 <link name="right_servo_1">
   <inertial>
-    <origin xyz="-0.008868375307288748 -0.01694602119485174 0.0048189227637153095" rpy="0 0 0"/>
+    <origin xyz="0.016946033965199135 -0.008868786547698113 0.0048191214240031685" rpy="0 0 0"/>
     <mass value="0.27778201352216375"/>
-    <inertia ixx="6.3e-05" iyy="6.8e-05" izz="3.8e-05" ixy="-4e-06" iyz="-1e-06" ixz="-1e-06"/>
-  </inertial>
-  <visual>
-    <origin xyz="0.069608 0.028345 -0.0235" rpy="0 0 0"/>
+    <inertia ixx="6.8e-05" iyy="6.3e-05" izz="3.8e-05" ixy="4e-06" iyz="-1e-06" ixz="1e-06"/>
+  </inertial>
+  <visual>
+    <origin xyz="-0.034659 0.063359 -0.021333" rpy="0 0 0"/>
     <geometry>
       <mesh filename="file://$(find leremix_description)/meshes/right_servo_1.stl" scale="0.001 0.001 0.001"/>
@@ -316,5 +316,5 @@
   </visual>
   <collision>
-    <origin xyz="0.069608 0.028345 -0.0235" rpy="0 0 0"/>
+    <origin xyz="-0.034659 0.063359 -0.021333" rpy="0 0 0"/>
     <geometry>
       <mesh filename="file://$(find leremix_description)/meshes/right_servo_1.stl" scale="0.001 0.001 0.001"/>
@@ -324,10 +324,10 @@
 <link name="right_wheel_mount_1">
   <inertial>
-    <origin xyz="-0.004783376671253933 -0.0027610611196918697 4.4100333345190035e-07" rpy="0 0 0"/>
+    <origin xyz="0.002761073890032273 -0.004782787911662353 -3.6033637842991517e-07" rpy="0 0 0"/>
     <mass value="0.1235708646349694"/>
-    <inertia ixx="2.9e-05" iyy="2.2e-05" izz="1.8e-05" ixy="6e-06" iyz="-0.0" ixz="0.0"/>
-  </inertial>
-  <visual>
-    <origin xyz="0.093574 0.054034 -0.015217" rpy="0 0 0"/>
+    <inertia ixx="2.2e-05" iyy="2.9e-05" izz="1.8e-05" ixy="-6e-06" iyz="0.0" ixz="0.0"/>
+  </inertial>
+  <visual>
+    <origin xyz="-0.060348 0.087326 -0.013051" rpy="0 0 0"/>
     <geometry>
       <mesh filename="file://$(find leremix_description)/meshes/right_wheel_mount_1.stl" scale="0.001 0.001 0.001"/>
@@ -336,5 +336,5 @@
   </visual>
   <collision>
-    <origin xyz="0.093574 0.054034 -0.015217" rpy="0 0 0"/>
+    <origin xyz="-0.060348 0.087326 -0.013051" rpy="0 0 0"/>
     <geometry>
       <mesh filename="file://$(find leremix_description)/meshes/right_wheel_mount_1.stl" scale="0.001 0.001 0.001"/>
@@ -344,10 +344,10 @@
 <link name="back_servo_mount_1">
   <inertial>
-    <origin xyz="0.02000689833996745 -0.015077228306122958 0.023640084058171418" rpy="0 0 0"/>
+    <origin xyz="0.015077241076461259 0.02000648709955183 0.023640282718459048" rpy="0 0 0"/>
     <mass value="0.13962178083501173"/>
-    <inertia ixx="4.7e-05" iyy="6.6e-05" izz="5e-05" ixy="0.0" iyz="2e-06" ixz="0.0"/>
-  </inertial>
-  <visual>
-    <origin xyz="0.02 -0.1 -0.005" rpy="0 0 0"/>
+    <inertia ixx="6.6e-05" iyy="4.7e-05" izz="5e-05" ixy="-0.0" iyz="0.0" ixz="-2e-06"/>
+  </inertial>
+  <visual>
+    <origin xyz="0.093686 0.013751 -0.002833" rpy="0 0 0"/>
     <geometry>
       <mesh filename="file://$(find leremix_description)/meshes/back_servo_mount_1.stl" scale="0.001 0.001 0.001"/>
@@ -356,5 +356,5 @@
   </visual>
   <collision>
-    <origin xyz="0.02 -0.1 -0.005" rpy="0 0 0"/>
+    <origin xyz="0.093686 0.013751 -0.002833" rpy="0 0 0"/>
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
File: ros/src/leremix_gazebo/urdf/gazebo_plugins.xacro (robot description, xacro)
@@ -7,5 +7,5 @@
             </plugin>
     </gazebo>
-    <gazebo reference="camera_1">
+    <gazebo reference="head_camera_1">
         <sensor type="camera" name="rgb_camera">
             <update_rate>30</update_rate>
@@ -28,5 +28,26 @@
         </sensor>
     </gazebo>
-    <gazebo reference="camera_1">
+        <gazebo reference="wrist_camera_v1_1">
+        <sensor type="camera" name="rgb_camera">
+            <update_rate>30</update_rate>
+            <camera name="head_rgb">
+            <horizontal_fov>1.0472</horizontal_fov> <!-- ~60 deg -->
+            <image>
+                <width>640</width>
+                <height>480</height>
+                <format>R8G8B8</format>
+            </image>
+            <clip>
+                <near>0.05</near>
+                <far>20.0</far>
+            </clip>
+            </camera>
+            <plugin name="gazebo_ros_camera" filename="libgazebo_ros_camera.so">
+                <namespace>/sensors/wrist_camera</namespace>
+                <frame_name>wrist_camera</frame_name>
+            </plugin>
+        </sensor>
+    </gazebo>
+    <gazebo reference="head_camera_1">
         <sensor type="depth" name="rgbd_camera">
             <update_rate>30</update_rate>
@@ -78,5 +99,5 @@
         </sensor>
     </gazebo>
-    <gazebo reference="camera_1">
+    <gazebo reference="lidar_1">
         <sensor name="lidar" type="ray">
             <always_on>true</always_on>
