Commit message: added fixes for simulation

File: ros/src/leremix_description/urdf/LeRemix.xacro (robot description, xacro)
@@ -2,9 +2,18 @@
 <robot name="LeRemix" xmlns:xacro="http://www.ros.org/wiki/xacro">
 <xacro:include filename="$(find leremix_description)/urdf/materials.xacro" />
+<!-- Empty root link for Gazebo compatibility -->
 <link name="base_link">
+</link>
+<!-- Fixed joint to actual base -->
+<joint name="robot_base_joint" type="fixed">
+  <origin xyz="0 0 0" rpy="0 0 0"/>
+  <parent link="base_link"/>
+  <child link="robot_base"/>
+</joint>
+<link name="robot_base">
   <inertial>
     <origin xyz="5.866413998148801e-05 0.0062819967824381704 0.001416599330144379" rpy="0 0 0"/>
-    <mass value="0.8949198281645031"/>
-    <inertia ixx="0.003064" iyy="0.002933" izz="0.005996" ixy="-2e-06" iyz="0.0" ixz="0.0"/>
+    <mass value="3.24"/>  <!-- base(440g) + battery(800g) -->
+    <inertia ixx="0.012" iyy="0.015" izz="0.020" ixy="-3.5e-06" iyz="0.0" ixz="0.0"/>
   </inertial>
   <visual>
@@ -13,5 +22,5 @@
       <mesh filename="file://$(find leremix_description)/meshes/base_link.stl" scale="0.001 0.001 0.001"/>
     </geometry>
-    <material name="silver"/>
+    <material name="Gazebo/DarkGrey"/>
   </visual>
   <collision>
@@ -25,6 +34,6 @@
   <inertial>
     <origin xyz="0.019999044959765788 0.01025034011227997 0.016027263585011595" rpy="0 0 0"/>
-    <mass value="0.2843033831904074"/>
-    <inertia ixx="4e-05" iyy="7.3e-05" izz="6.2e-05" ixy="0.0" iyz="0.0" ixz="-1e-06"/>
+    <mass value="0.05"/>  <!-- ST3215 servo 50g -->
+    <inertia ixx="2.1e-05" iyy="4.2e-05" izz="3.5e-05" ixy="0.0" iyz="0.0" ixz="-1e-06"/>
   </inertial>
   <visual>
@@ -33,5 +42,5 @@
       <mesh filename="file://$(find leremix_description)/meshes/arm_base_rotation_servo_1.stl" scale="0.001 0.001 0.001"/>
     </geometry>
-    <material name="silver"/>
+    <material name="Gazebo/DarkGrey"/>
   </visual>
   <collision>
@@ -45,6 +54,6 @@
   <inertial>
     <origin xyz="0.03155588382289583 -0.00027122946045804366 -0.009540250989642243" rpy="0 0 0"/>
-    <mass value="0.5385469320676795"/>
-    <inertia ixx="0.000341" iyy="0.000375" izz="0.000154" ixy="-1e-06" iyz="3e-06" ixz="-3.6e-05"/>
+    <mass value="0.03"/>  <!-- Arm plastic part -->
+    <inertia ixx="1.2e-04" iyy="1.5e-04" izz="8.0e-05" ixy="-9e-08" iyz="3e-07" ixz="-3.3e-06"/>
   </inertial>
   <visual>
@@ -53,5 +62,5 @@
       <mesh filename="file://$(find leremix_description)/meshes/arm_base_rotation_link_1.stl" scale="0.001 0.001 0.001"/>
     </geometry>
-    <material name="silver"/>
+    <material name="Gazebo/DarkGrey"/>
   </visual>
   <collision>
@@ -65,6 +74,6 @@
   <inertial>
     <origin xyz="-0.009494213831683473 0.023250133340888265 -0.002658011177624875" rpy="0 0 0"/>
-    <mass value="0.10853073755546007"/>
-    <inertia ixx="4.6e-05" iyy="2.7e-05" izz="5.8e-05" ixy="-0.0" iyz="-0.0" ixz="-0.0"/>
+    <mass value="0.015"/>  <!-- Small plastic cover -->
+    <inertia ixx="2.5e-05" iyy="1.8e-05" izz="3.2e-05" ixy="-0.0" iyz="-0.0" ixz="-0.0"/>
   </inertial>
   <visual>
@@ -73,5 +82,5 @@
       <mesh filename="file://$(find leremix_description)/meshes/arm_base_rotation_link_cover_1.stl" scale="0.001 0.001 0.001"/>
     </geometry>
-    <material name="silver"/>
+    <material name="Gazebo/DarkGrey"/>
   </visual>
   <collision>
@@ -85,6 +94,6 @@
   <inertial>
     <origin xyz="-0.010249982610195635 -0.016026724819197403 0.019999226223505806" rpy="0 0 0"/>
-    <mass value="0.2843033831904074"/>
-    <inertia ixx="7.3e-05" iyy="6.2e-05" izz="4e-05" ixy="0.0" iyz="1e-06" ixz="-0.0"/>
+    <mass value="0.05"/>  <!-- ST3215 servo 50g -->
+    <inertia ixx="2.1e-05" iyy="3.5e-05" izz="4.2e-05" ixy="0.0" iyz="1e-07" ixz="-0.0"/>
   </inertial>
   <visual>
@@ -93,5 +102,5 @@
       <mesh filename="file://$(find leremix_description)/meshes/arm_shoulder_servo_1.stl" scale="0.001 0.001 0.001"/>
     </geometry>
-    <material name="silver"/>
+    <material name="Gazebo/DarkGrey"/>
   </visual>
   <collision>
@@ -105,6 +114,6 @@
   <inertial>
     <origin xyz="-0.055943188746678085 0.01969986419355535 -0.015368056226457844" rpy="0 0 0"/>
-    <mass value="0.9906249126045027"/>
-    <inertia ixx="0.000563" iyy="0.001251" izz="0.001549" ixy="-8e-06" iyz="-3e-06" ixz="-0.000304"/>
+    <mass value="0.04"/>  <!-- Arm plastic link -->
+    <inertia ixx="1.2e-04" iyy="2.5e-04" izz="3.0e-04" ixy="-4e-07" iyz="-2e-07" ixz="-1.5e-05"/>
   </inertial>
   <visual>
@@ -113,5 +122,5 @@
       <mesh filename="file://$(find leremix_description)/meshes/arm_shoulder_link_1.stl" scale="0.001 0.001 0.001"/>
     </geometry>
-    <material name="silver"/>
+    <material name="Gazebo/DarkGrey"/>
   </visual>
   <collision>
@@ -125,6 +134,6 @@
   <inertial>
     <origin xyz="-0.015077029653089111 -0.016026724819193545 0.016665077642131626" rpy="0 0 0"/>
-    <mass value="0.2843033831904074"/>
-    <inertia ixx="7.1e-05" iyy="6.2e-05" izz="4.2e-05" ixy="-0.0" iyz="1e-06" ixz="8e-06"/>
+    <mass value="0.05"/>  <!-- ST3215 servo 50g -->
+    <inertia ixx="2.5e-05" iyy="3.5e-05" izz="4.4e-05" ixy="-0.0" iyz="1e-07" ixz="8e-07"/>
   </inertial>
   <visual>
@@ -133,5 +142,5 @@
       <mesh filename="file://$(find leremix_description)/meshes/arm_elbow_servo_1.stl" scale="0.001 0.001 0.001"/>
     </geometry>
-    <material name="silver"/>
+    <material name="Gazebo/DarkGrey"/>
   </visual>
   <collision>
@@ -145,6 +154,6 @@
   <inertial>
     <origin xyz="0.05832613508152747 0.015215218913568064 0.02137713488564641" rpy="0 0 0"/>
-    <mass value="0.8772447501056027"/>
-    <inertia ixx="0.000473" iyy="0.000993" izz="0.001135" ixy="-0.000109" iyz="-4.1e-05" ixz="-0.000289"/>
+    <mass value="0.04"/>
+    <inertia ixx="2.2e-05" iyy="4.5e-05" izz="5.2e-05" ixy="-5e-06" iyz="-1.9e-06" ixz="-1.3e-05"/>
   </inertial>
   <visual>
@@ -153,5 +162,5 @@
       <mesh filename="file://$(find leremix_description)/meshes/arm_elbow_link_1.stl" scale="0.001 0.001 0.001"/>
     </geometry>
-    <material name="silver"/>
+    <material name="Gazebo/DarkGrey"/>
   </visual>
   <collision>
@@ -165,6 +174,6 @@
   <inertial>
     <origin xyz="0.021970231163924825 -0.016026724819192876 -0.004724278591325293" rpy="0 0 0"/>
-    <mass value="0.2843033831904074"/>
-    <inertia ixx="4.2e-05" iyy="6.2e-05" izz="7.1e-05" ixy="1e-06" iyz="0.0" ixz="-8e-06"/>
+    <mass value="0.05"/>  <!-- ST3215 servo 50g -->
+    <inertia ixx="4.4e-05" iyy="3.5e-05" izz="2.5e-05" ixy="1e-07" iyz="0.0" ixz="-8e-07"/>
   </inertial>
   <visual>
@@ -173,5 +182,5 @@
       <mesh filename="file://$(find leremix_description)/meshes/arm_wrist_tilt_servo_1.stl" scale="0.001 0.001 0.001"/>
     </geometry>
-    <material name="silver"/>
+    <material name="Gazebo/DarkGrey"/>
   </visual>
   <collision>
@@ -185,6 +194,6 @@
   <inertial>
     <origin xyz="0.012975594362619927 0.016810121377602565 -0.02296834504128556" rpy="0 0 0"/>
-    <mass value="0.2392168278135931"/>
-    <inertia ixx="0.000182" iyy="0.000115" izz="0.000144" ixy="3e-06" iyz="-6e-06" ixz="3.2e-05"/>
+    <mass value="0.02"/>
+    <inertia ixx="1.5e-05" iyy="9.6e-06" izz="1.2e-05" ixy="3e-07" iyz="-5e-07" ixz="2.7e-06"/>
   </inertial>
   <visual>
@@ -193,5 +202,5 @@
       <mesh filename="file://$(find leremix_description)/meshes/arm_wrist_link_1.stl" scale="0.001 0.001 0.001"/>
     </geometry>
-    <material name="silver"/>
+    <material name="Gazebo/DarkGrey"/>
   </visual>
   <collision>
@@ -205,6 +214,6 @@
   <inertial>
     <origin xyz="-0.01656958325728916 0.015998644972749377 0.008429716426542305" rpy="0 0 0"/>
-    <mass value="0.2799142523131049"/>
-    <inertia ixx="6.9e-05" iyy="3.8e-05" izz="6.3e-05" ixy="-1e-06" iyz="1e-06" ixz="5e-06"/>
+    <mass value="0.05"/>  <!-- ST3215 servo 50g -->
+    <inertia ixx="2.4e-05" iyy="4.1e-05" izz="3.8e-05" ixy="-1e-07" iyz="1e-07" ixz="5e-07"/>
   </inertial>
   <visual>
@@ -213,5 +222,5 @@
       <mesh filename="file://$(find leremix_description)/meshes/arm_wrist_roll_servo_1.stl" scale="0.001 0.001 0.001"/>
     </geometry>
-    <material name="silver"/>
+    <material name="Gazebo/DarkGrey"/>
   </visual>
   <collision>
@@ -225,6 +234,6 @@
   <inertial>
     <origin xyz="0.013339671966003358 -0.013714806926169776 -0.026125553965198" rpy="0 0 0"/>
-    <mass value="0.44698022927880193"/>
-    <inertia ixx="0.000294" iyy="0.000301" izz="0.000205" ixy="3e-05" iyz="-4.7e-05" ixz="7.1e-05"/>
+    <mass value="0.02"/>
+    <inertia ixx="1.3e-05" iyy="1.3e-05" izz="9.2e-06" ixy="1.3e-06" iyz="-2.1e-06" ixz="3.2e-06"/>
   </inertial>
   <visual>
@@ -233,5 +242,5 @@
       <mesh filename="file://$(find leremix_description)/meshes/arm_gripper_1.stl" scale="0.001 0.001 0.001"/>
     </geometry>
-    <material name="silver"/>
+    <material name="Gazebo/DarkGrey"/>
   </visual>
   <collision>
@@ -245,6 +254,6 @@
   <inertial>
     <origin xyz="-0.007975468163954197 0.020789656863227802 -0.01631207348591407" rpy="0 0 0"/>
-    <mass value="0.2843033831904074"/>
-    <inertia ixx="6.4e-05" iyy="4e-05" izz="7.1e-05" ixy="-0.0" iyz="-0.0" ixz="-5e-06"/>
+    <mass value="0.05"/>  <!-- ST3215 servo 50g -->
+    <inertia ixx="3.7e-05" iyy="4.2e-05" izz="2.5e-05" ixy="-0.0" iyz="-0.0" ixz="-5e-07"/>
   </inertial>
   <visual>
@@ -253,5 +262,5 @@
       <mesh filename="file://$(find leremix_description)/meshes/arm_gripper_servo_1.stl" scale="0.001 0.001 0.001"/>
     </geometry>
-    <material name="silver"/>
+    <material name="Gazebo/DarkGrey"/>
   </visual>
   <collision>
@@ -265,6 +274,6 @@
   <inertial>
     <origin xyz="0.032905631581261585 -0.003660190112443975 -0.016197173267020665" rpy="0 0 0"/>
-    <mass value="0.1586808414280307"/>
-    <inertia ixx="6.1e-05" iyy="8.6e-05" izz="3.4e-05" ixy="4e-06" iyz="-5e-06" ixz="1.9e-05"/>
+    <mass value="0.01"/>
+    <inertia ixx="3.8e-06" iyy="5.4e-06" izz="2.1e-06" ixy="3e-07" iyz="-3e-07" ixz="1.2e-06"/>
   </inertial>
   <visual>
@@ -273,5 +282,5 @@
       <mesh filename="file://$(find leremix_description)/meshes/arm_jaw_1.stl" scale="0.001 0.001 0.001"/>
     </geometry>
-    <material name="silver"/>
+    <material name="Gazebo/DarkGrey"/>
   </visual>
   <collision>
@@ -285,6 +294,6 @@
   <inertial>
     <origin xyz="0.02008674389712354 0.005193645092054736 0.023611795909587813" rpy="0 0 0"/>
-    <mass value="0.14423806644766202"/>
-    <inertia ixx="5.5e-05" iyy="6.4e-05" izz="5.3e-05" ixy="-8e-06" iyz="-1e-06" ixz="1e-06"/>
+    <mass value="0.05"/>
+    <inertia ixx="1.9e-05" iyy="2.2e-05" izz="1.8e-05" ixy="-3e-06" iyz="-3e-07" ixz="3e-07"/>
   </inertial>
   <visual>
@@ -293,5 +302,5 @@
       <mesh filename="file://$(find leremix_description)/meshes/right_servo_mount_1.stl" scale="0.001 0.001 0.001"/>
     </geometry>
-    <material name="silver"/>
+    <material name="Gazebo/DarkGrey"/>
   </visual>
   <collision>
@@ -305,6 +314,6 @@
   <inertial>
     <origin xyz="0.016946033965199135 -0.008868786547698113 0.0048191214240031685" rpy="0 0 0"/>
-    <mass value="0.27778201352216375"/>
-    <inertia ixx="6.8e-05" iyy="6.3e-05" izz="3.8e-05" ixy="4e-06" iyz="-1e-06" ixz="1e-06"/>
+    <mass value="0.05"/>  <!-- ST3215 servo 50g -->
+    <inertia ixx="2.3e-05" iyy="3.8e-05" izz="4.1e-05" ixy="4e-07" iyz="-1e-07" ixz="1e-07"/>
   </inertial>
   <visual>
@@ -313,5 +322,5 @@
       <mesh filename="file://$(find leremix_description)/meshes/right_servo_1.stl" scale="0.001 0.001 0.001"/>
     </geometry>
-    <material name="silver"/>
+    <material name="Gazebo/DarkGrey"/>
   </visual>
   <collision>
@@ -325,6 +334,6 @@
   <inertial>
     <origin xyz="0.002761073890032273 -0.004782787911662353 -3.6033637842991517e-07" rpy="0 0 0"/>
-    <mass value="0.1235708646349694"/>
-    <inertia ixx="2.2e-05" iyy="2.9e-05" izz="1.8e-05" ixy="-6e-06" iyz="0.0" ixz="0.0"/>
+    <mass value="0.05"/>
+    <inertia ixx="8.9e-06" iyy="1.2e-05" izz="7.3e-06" ixy="-2.4e-06" iyz="0.0" ixz="0.0"/>
   </inertial>
   <visual>
@@ -333,5 +342,5 @@
       <mesh filename="file://$(find leremix_description)/meshes/right_wheel_mount_1.stl" scale="0.001 0.001 0.001"/>
     </geometry>
-    <material name="silver"/>
+    <material name="Gazebo/DarkGrey"/>
   </visual>
   <collision>
@@ -345,6 +354,6 @@
   <inertial>
     <origin xyz="0.015077241076461259 0.02000648709955183 0.023640282718459048" rpy="0 0 0"/>
-    <mass value="0.13962178083501173"/>
-    <inertia ixx="6.6e-05" iyy="4.7e-05" izz="5e-05" ixy="-0.0" iyz="0.0" ixz="-2e-06"/>
+    <mass value="0.05"/>
+    <inertia ixx="2.4e-05" iyy="1.7e-05" izz="1.8e-05" ixy="-0.0" iyz="0.0" ixz="-7e-07"/>
   </inertial>
   <visual>
@@ -353,5 +362,5 @@
       <mesh filename="file://$(find leremix_description)/meshes/back_servo_mount_1.stl" scale="0.001 0.001 0.001"/>
     </geometry>
-    <material name="silver"/>
+    <material name="Gazebo/DarkGrey"/>
   </visual>
   <collision>
@@ -365,6 +374,6 @@
   <inertial>
     <origin xyz="0.009786012594139637 -0.023059797468141602 0.023640282726657757" rpy="0 0 0"/>
-    <mass value="0.13962178077674334"/>
-    <inertia ixx="5.2e-05" iyy="6.2e-05" izz="5e-05" ixy="8e-06" iyz="1e-06" ixz="1e-06"/>
+    <mass value="0.05"/>
+    <inertia ixx="1.9e-05" iyy="2.2e-05" izz="1.8e-05" ixy="3e-06" iyz="4e-07" ixz="4e-07"/>
   </inertial>
   <visual>
@@ -373,5 +382,5 @@
       <mesh filename="file://$(find leremix_description)/meshes/left_servo_mount_1.stl" scale="0.001 0.001 0.001"/>
     </geometry>
-    <material name="silver"/>
+    <material name="Gazebo/DarkGrey"/>
   </visual>
   <collision>
@@ -385,6 +394,6 @@
   <inertial>
     <origin xyz="-0.016153032440181764 -0.010249777894134756 -0.019698916271482823" rpy="0 0 0"/>
-    <mass value="0.2777820135235829"/>
-    <inertia ixx="6e-05" iyy="7e-05" izz="3.8e-05" ixy="-0.0" iyz="-0.0" ixz="-1e-06"/>
+    <mass value="0.05"/>  <!-- ST3215 servo 50g -->
+    <inertia ixx="3.5e-05" iyy="2.5e-05" izz="4.1e-05" ixy="-0.0" iyz="-0.0" ixz="-1e-07"/>
   </inertial>
   <visual>
@@ -393,5 +402,5 @@
       <mesh filename="file://$(find leremix_description)/meshes/back_servo_1.stl" scale="0.001 0.001 0.001"/>
     </geometry>
-    <material name="silver"/>
+    <material name="Gazebo/DarkGrey"/>
   </visual>
   <collision>
@@ -405,6 +414,6 @@
   <inertial>
     <origin xyz="0.007687527486229681 -0.0133147596761716 -4.2527541098749677e-07" rpy="0 0 0"/>
-    <mass value="1.3542854082324305"/>
-    <inertia ixx="0.00129" iyy="0.001683" izz="0.001094" ixy="-0.00034" iyz="-0.0" ixz="-0.0"/>
+    <mass value="0.32"/>  <!-- 320g omni wheel -->
+    <inertia ixx="0.0008" iyy="0.0012" izz="0.0008" ixy="-8e-05" iyz="-0.0" ixz="-0.0"/>
   </inertial>
   <visual>
@@ -413,5 +422,5 @@
       <mesh filename="file://$(find leremix_description)/meshes/right_wheel_1.stl" scale="0.001 0.001 0.001"/>
     </geometry>
-    <material name="silver"/>
+    <material name="Gazebo/DarkGrey"/>
   </visual>
   <collision>
@@ -425,6 +434,6 @@
   <inertial>
     <origin xyz="-0.00552250463639424 2.1693908731044986e-07 -4.169788832414367e-07" rpy="0 0 0"/>
-    <mass value="0.1235708646349694"/>
-    <inertia ixx="3.3e-05" iyy="1.8e-05" izz="1.8e-05" ixy="-0.0" iyz="-0.0" ixz="-0.0"/>
+    <mass value="0.05"/>
+    <inertia ixx="1.3e-05" iyy="7.3e-06" izz="7.3e-06" ixy="-0.0" iyz="-0.0" ixz="-0.0"/>
   </inertial>
   <visual>
@@ -433,5 +442,5 @@
       <mesh filename="file://$(find leremix_description)/meshes/back_wheel_mount_1.stl" scale="0.001 0.001 0.001"/>
     </geometry>
-    <material name="silver"/>
+    <material name="Gazebo/DarkGrey"/>
   </visual>
   <collision>
@@ -445,6 +454,6 @@
   <inertial>
     <origin xyz="-0.015374617586046052 1.0825471297073314e-07 -3.3995992976439127e-07" rpy="0 0 0"/>
-    <mass value="1.3542854082324305"/>
-    <inertia ixx="0.00188" iyy="0.001094" izz="0.001094" ixy="0.0" iyz="0.0" ixz="-0.0"/>
+    <mass value="0.32"/>  <!-- 320g omni wheel -->
+    <inertia ixx="0.0012" iyy="0.0008" izz="0.0008" ixy="0.0" iyz="0.0" ixz="-0.0"/>
   </inertial>
   <visual>
@@ -453,5 +462,5 @@
       <mesh filename="file://$(find leremix_description)/meshes/back_wheel_1.stl" scale="0.001 0.001 0.001"/>
     </geometry>
-    <material name="silver"/>
+    <material name="Gazebo/DarkGrey"/>
   </visual>
   <collision>
@@ -465,6 +474,6 @@
   <inertial>
     <origin xyz="0.016924848422785556 0.00888142204280122 -0.019716322743522894" rpy="0 0 0"/>
-    <mass value="0.27778201352216375"/>
-    <inertia ixx="6.8e-05" iyy="6.3e-05" izz="3.8e-05" ixy="-4e-06" iyz="1e-06" ixz="0.0"/>
+    <mass value="0.05"/>  <!-- ST3215 servo 50g -->
+    <inertia ixx="2.3e-05" iyy="3.8e-05" izz="4.1e-05" ixy="-4e-07" iyz="1e-07" ixz="0.0"/>
   </inertial>
   <visual>
@@ -473,5 +482,5 @@
       <mesh filename="file://$(find leremix_description)/meshes/left_servo_1.stl" scale="0.001 0.001 0.001"/>
     </geometry>
-    <material name="silver"/>
+    <material name="Gazebo/DarkGrey"/>
   </visual>
   <collision>
@@ -485,6 +494,6 @@
   <inertial>
     <origin xyz="0.002761280694251654 0.004782713545836703 1.954960941463746e-07" rpy="0 0 0"/>
-    <mass value="0.1235708646349694"/>
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