Commit message: added fixes for simulation

File: ros/src/leremix_gazebo/urdf/gazebo_configs.xacro (robot description, xacro)
@@ -3,253 +3,316 @@
   <max_step_size>0.001</max_step_size>
   <real_time_update_rate>1000</real_time_update_rate>
+   <ode>
+    <solver type="quick" iters="150" sor="1.3"/>
+    <constraints cfm="0.0" erp="0.2"
+      contact_max_correcting_vel="0.5"
+      contact_surface_layer="0.001"/>
+  </ode>
+</physics>
+<physics type="ode">
+  <max_step_size>0.001</max_step_size>
+  <real_time_update_rate>1000</real_time_update_rate>
   <ode>
-    <solver><type>quick</type><iters>80</iters><sor>1.2</sor></solver>
-    <constraints>
-      <cfm>1e-5</cfm><erp>0.2</erp>
-      <contact_max_correcting_vel>30.0</contact_max_correcting_vel>
-      <contact_surface_layer>0.002</contact_surface_layer>
-    </constraints>
+    <solver type="quick" iters="150" sor="1.3"/>
+    <constraints cfm="0.0" erp="0.2"
+      contact_max_correcting_vel="0.5"
+      contact_surface_layer="0.001"/>
   </ode>
 </physics>
 <gazebo reference="base_link">
-  <mu1>0.2</mu1>
-  <mu2>0.2</mu2>
-  <self_collide>true</self_collide>
+  <material>Gazebo/FlatBlack</material>
+  <mu1>0.2</mu1>
+  <mu2>0.2</mu2>
+  <self_collide>false</self_collide>
   <gravity>true</gravity>
 </gazebo>
+<gazebo reference="robot_base">
+  <material>Gazebo/FlatBlack</material>
+  <mu1>0.2</mu1>
+  <mu2>0.2</mu2>
+  <self_collide>false</self_collide>
+  <gravity>true</gravity>
+</gazebo>
 <gazebo reference="arm_base_rotation_servo_1">
-  <mu1>0.2</mu1>
-  <mu2>0.2</mu2>
-  <self_collide>true</self_collide>
+  <material>Gazebo/White</material>
+  <mu1>0.2</mu1>
+  <mu2>0.2</mu2>
+  <self_collide>false</self_collide>
 </gazebo>
 <gazebo reference="arm_base_rotation_link_1">
-  <mu1>0.2</mu1>
-  <mu2>0.2</mu2>
-  <self_collide>true</self_collide>
+  <material>Gazebo/DarkGrey</material>
+  <mu1>0.2</mu1>
+  <mu2>0.2</mu2>
+  <self_collide>false</self_collide>
 </gazebo>
 <gazebo reference="arm_base_rotation_link_cover_1">
-  <mu1>0.2</mu1>
-  <mu2>0.2</mu2>
-  <self_collide>true</self_collide>
+  <material>Gazebo/DarkGrey</material>
+  <mu1>0.2</mu1>
+  <mu2>0.2</mu2>
+  <self_collide>false</self_collide>
 </gazebo>
 <gazebo reference="arm_shoulder_servo_1">
-  <mu1>0.2</mu1>
-  <mu2>0.2</mu2>
-  <self_collide>true</self_collide>
+  <material>Gazebo/White</material>
+  <mu1>0.2</mu1>
+  <mu2>0.2</mu2>
+  <self_collide>false</self_collide>
 </gazebo>
 <gazebo reference="arm_shoulder_link_1">
-  <mu1>0.2</mu1>
-  <mu2>0.2</mu2>
-  <self_collide>true</self_collide>
+  <material>Gazebo/DarkGrey</material>
+  <mu1>0.2</mu1>
+  <mu2>0.2</mu2>
+  <self_collide>false</self_collide>
 </gazebo>
 <gazebo reference="arm_elbow_servo_1">
-  <mu1>0.2</mu1>
-  <mu2>0.2</mu2>
-  <self_collide>true</self_collide>
+  <material>Gazebo/White</material>
+  <mu1>0.2</mu1>
+  <mu2>0.2</mu2>
+  <self_collide>false</self_collide>
 </gazebo>
 <gazebo reference="arm_elbow_link_1">
-  <mu1>0.2</mu1>
-  <mu2>0.2</mu2>
-  <self_collide>true</self_collide>
+  <material>Gazebo/DarkGrey</material>
+  <mu1>0.2</mu1>
+  <mu2>0.2</mu2>
+  <self_collide>false</self_collide>
 </gazebo>
 <gazebo reference="arm_wrist_tilt_servo_1">
-  <mu1>0.2</mu1>
-  <mu2>0.2</mu2>
-  <self_collide>true</self_collide>
+  <material>Gazebo/White</material>
+  <mu1>0.2</mu1>
+  <mu2>0.2</mu2>
+  <self_collide>false</self_collide>
 </gazebo>
 <gazebo reference="arm_wrist_link_1">
-  <mu1>0.2</mu1>
-  <mu2>0.2</mu2>
-  <self_collide>true</self_collide>
+  <material>Gazebo/DarkGrey</material>
+  <mu1>0.2</mu1>
+  <mu2>0.2</mu2>
+  <self_collide>false</self_collide>
 </gazebo>
 <gazebo reference="arm_wrist_roll_servo_1">
-  <mu1>0.2</mu1>
-  <mu2>0.2</mu2>
-  <self_collide>true</self_collide>
+  <material>Gazebo/White</material>
+  <mu1>0.2</mu1>
+  <mu2>0.2</mu2>
+  <self_collide>false</self_collide>
 </gazebo>
 <gazebo reference="arm_gripper_1">
-  <mu1>0.2</mu1>
-  <mu2>0.2</mu2>
-  <self_collide>true</self_collide>
+  <material>Gazebo/DarkGrey</material>
+  <mu1>0.2</mu1>
+  <mu2>0.2</mu2>
+  <self_collide>false</self_collide>
 </gazebo>
 <gazebo reference="arm_gripper_servo_1">
-  <mu1>0.2</mu1>
-  <mu2>0.2</mu2>
-  <self_collide>true</self_collide>
+  <material>Gazebo/White</material>
+  <mu1>0.2</mu1>
+  <mu2>0.2</mu2>
+  <self_collide>false</self_collide>
 </gazebo>
 <gazebo reference="arm_jaw_1">
-  <mu1>0.2</mu1>
-  <mu2>0.2</mu2>
-  <self_collide>true</self_collide>
+  <material>Gazebo/DarkGrey</material>
+  <mu1>0.2</mu1>
+  <mu2>0.2</mu2>
+  <self_collide>false</self_collide>
 </gazebo>
 <gazebo reference="right_servo_mount_1">
-  <mu1>0.2</mu1>
-  <mu2>0.2</mu2>
-  <self_collide>true</self_collide>
+  <material>Gazebo/DarkGrey</material>
+  <mu1>0.2</mu1>
+  <mu2>0.2</mu2>
+  <self_collide>false</self_collide>
 </gazebo>
 <gazebo reference="right_servo_1">
-  <mu1>0.2</mu1>
-  <mu2>0.2</mu2>
-  <self_collide>true</self_collide>
+  <material>Gazebo/White</material>
+  <mu1>0.2</mu1>
+  <mu2>0.2</mu2>
+  <self_collide>false</self_collide>
 </gazebo>
 <gazebo reference="back_servo_mount_1">
-  <mu1>0.2</mu1>
-  <mu2>0.2</mu2>
-  <self_collide>true</self_collide>
+  <material>Gazebo/DarkGrey</material>
+  <mu1>0.2</mu1>
+  <mu2>0.2</mu2>
+  <self_collide>false</self_collide>
 </gazebo>
 <gazebo reference="left_servo_mount_1">
-  <mu1>0.2</mu1>
-  <mu2>0.2</mu2>
-  <self_collide>true</self_collide>
+  <material>Gazebo/DarkGrey</material>
+  <mu1>0.2</mu1>
+  <mu2>0.2</mu2>
+  <self_collide>false</self_collide>
 </gazebo>
 <gazebo reference="back_servo_1">
-  <mu1>0.2</mu1>
-  <mu2>0.2</mu2>
-  <self_collide>true</self_collide>
+  <material>Gazebo/White</material>
+  <mu1>0.2</mu1>
+  <mu2>0.2</mu2>
+  <self_collide>false</self_collide>
 </gazebo>
 <gazebo reference="back_wheel_mount_1">
-  <mu1>0.2</mu1>
-  <mu2>0.2</mu2>
-  <self_collide>true</self_collide>
+  <material>Gazebo/DarkGrey</material>
+  <mu1>0.2</mu1>
+  <mu2>0.2</mu2>
+  <self_collide>false</self_collide>
 </gazebo>
 <gazebo reference="back_wheel_1">
-  <mu1>0.2</mu1>
-  <mu2>0.2</mu2>
-  <self_collide>true</self_collide>
+  <material>Gazebo/DarkGrey</material>
+  <mu1>0.2</mu1>
+  <mu2>0.2</mu2>
+  <self_collide>false</self_collide>
 </gazebo>
 <gazebo reference="left_servo_1">
-  <mu1>0.2</mu1>
-  <mu2>0.2</mu2>
-  <self_collide>true</self_collide>
+  <material>Gazebo/White</material>
+  <mu1>0.2</mu1>
+  <mu2>0.2</mu2>
+  <self_collide>false</self_collide>
 </gazebo>
 <gazebo reference="left_wheel_mount_1">
-  <mu1>0.2</mu1>
-  <mu2>0.2</mu2>
-  <self_collide>true</self_collide>
+  <material>Gazebo/DarkGrey</material>
+  <mu1>0.2</mu1>
+  <mu2>0.2</mu2>
+  <self_collide>false</self_collide>
 </gazebo>
 <gazebo reference="orin_1">
-  <mu1>0.2</mu1>
-  <mu2>0.2</mu2>
-  <self_collide>true</self_collide>
+  <material>Gazebo/Grey</material>
+  <mu1>0.2</mu1>
+  <mu2>0.2</mu2>
+  <self_collide>false</self_collide>
 </gazebo>
 <gazebo reference="orin_mount_1">
-  <mu1>0.2</mu1>
-  <mu2>0.2</mu2>
-  <self_collide>true</self_collide>
+  <material>Gazebo/DarkGrey</material>
+  <mu1>0.2</mu1>
+  <mu2>0.2</mu2>
+  <self_collide>false</self_collide>
 </gazebo>
 <gazebo reference="battery_stopper_1">
-  <mu1>0.2</mu1>
-  <mu2>0.2</mu2>
-  <self_collide>true</self_collide>
+  <material>Gazebo/DarkGrey</material>
+  <mu1>0.2</mu1>
+  <mu2>0.2</mu2>
+  <self_collide>false</self_collide>
 </gazebo>
 <gazebo reference="usb_pd_mount_1">
-  <mu1>0.2</mu1>
-  <mu2>0.2</mu2>
-  <self_collide>true</self_collide>
+  <material>Gazebo/DarkGrey</material>
+  <mu1>0.2</mu1>
+  <mu2>0.2</mu2>
+  <self_collide>false</self_collide>
 </gazebo>
 <gazebo reference="arm_base_1">
-  <mu1>0.2</mu1>
-  <mu2>0.2</mu2>
-  <self_collide>true</self_collide>
+  <material>Gazebo/DarkGrey</material>
+  <mu1>0.2</mu1>
+  <mu2>0.2</mu2>
+  <self_collide>false</self_collide>
 </gazebo>
 <gazebo reference="imu_1">
-  <mu1>0.2</mu1>
-  <mu2>0.2</mu2>
-  <self_collide>true</self_collide>
+  <material>Gazebo/Blue</material>
+  <mu1>0.2</mu1>
+  <mu2>0.2</mu2>
+  <self_collide>false</self_collide>
 </gazebo>
 <gazebo reference="imu_mount_1">
-  <mu1>0.2</mu1>
-  <mu2>0.2</mu2>
-  <self_collide>true</self_collide>
+  <material>Gazebo/DarkGrey</material>
+  <mu1>0.2</mu1>
+  <mu2>0.2</mu2>
+  <self_collide>false</self_collide>
 </gazebo>
 <gazebo reference="hex_1__1__1">
-  <mu1>0.2</mu1>
-  <mu2>0.2</mu2>
-  <self_collide>true</self_collide>
+  <material>Gazebo/DarkYellow</material>
+  <mu1>0.2</mu1>
+  <mu2>0.2</mu2>
+  <self_collide>false</self_collide>
 </gazebo>
 <gazebo reference="just_the_tower_v1_1">
-  <mu1>0.2</mu1>
-  <mu2>0.2</mu2>
-  <self_collide>true</self_collide>
+  <material>Gazebo/DarkGrey</material>
+  <mu1>0.2</mu1>
+  <mu2>0.2</mu2>
+  <self_collide>false</self_collide>
 </gazebo>
 <gazebo reference="support_v1_1">
-  <mu1>0.2</mu1>
-  <mu2>0.2</mu2>
-  <self_collide>true</self_collide>
+  <material>Gazebo/DarkGrey</material>
+  <mu1>0.2</mu1>
+  <mu2>0.2</mu2>
+  <self_collide>false</self_collide>
 </gazebo>
 <gazebo reference="head_camera_1">
-  <mu1>0.2</mu1>
-  <mu2>0.2</mu2>
-  <self_collide>true</self_collide>
+  <material>Gazebo/DarkGrey</material>
+  <mu1>0.2</mu1>
+  <mu2>0.2</mu2>
+  <self_collide>false</self_collide>
 </gazebo>
 <gazebo reference="hex_1_1">
-  <mu1>0.2</mu1>
-  <mu2>0.2</mu2>
-  <self_collide>true</self_collide>
+  <material>Gazebo/DarkYellow</material>
+  <mu1>0.2</mu1>
+  <mu2>0.2</mu2>
+  <self_collide>false</self_collide>
 </gazebo>
 <gazebo reference="hex_2_1">
-  <mu1>0.2</mu1>
-  <mu2>0.2</mu2>
-  <self_collide>true</self_collide>
+  <material>Gazebo/DarkYellow</material>
+  <mu1>0.2</mu1>
+  <mu2>0.2</mu2>
+  <self_collide>false</self_collide>
 </gazebo>
 <gazebo reference="hex_1__1___1__1">
-  <mu1>0.2</mu1>
-  <mu2>0.2</mu2>
-  <self_collide>true</self_collide>
+  <material>Gazebo/DarkYellow</material>
+  <mu1>0.2</mu1>
+  <mu2>0.2</mu2>
+  <self_collide>false</self_collide>
 </gazebo>
 <gazebo reference="last_floor_v1_1">
-  <mu1>0.2</mu1>
-  <mu2>0.2</mu2>
-  <self_collide>true</self_collide>
+  <material>Gazebo/FlatBlack</material>
+  <mu1>0.2</mu1>
+  <mu2>0.2</mu2>
+  <self_collide>false</self_collide>
 </gazebo>
 <gazebo reference="front_cam_support_1">
-  <mu1>0.2</mu1>
-  <mu2>0.2</mu2>
-  <self_collide>true</self_collide>
+  <material>Gazebo/DarkGrey</material>
+  <mu1>0.2</mu1>
+  <mu2>0.2</mu2>
+  <self_collide>false</self_collide>
 </gazebo>
 <gazebo reference="front_camera_1">
-  <mu1>0.2</mu1>
-  <mu2>0.2</mu2>
-  <self_collide>true</self_collide>
+  <material>Gazebo/Blue</material>
+  <mu1>0.2</mu1>
+  <mu2>0.2</mu2>
+  <self_collide>false</self_collide>
 </gazebo>
 <gazebo reference="hex_3_1">
-  <mu1>0.2</mu1>
-  <mu2>0.2</mu2>
-  <self_collide>true</self_collide>
+  <material>Gazebo/DarkYellow</material>
+  <mu1>0.2</mu1>
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
File: ros/src/leremix_gazebo/urdf/gazebo_plugins.xacro (robot description, xacro)
@@ -7,5 +7,5 @@
             </plugin>
     </gazebo>
-    <gazebo reference="head_camera_1">
+    <gazebo reference="head_camera_frame">
         <sensor type="camera" name="rgb_camera">
             <update_rate>30</update_rate>
@@ -23,10 +23,31 @@
             </camera>
             <plugin name="gazebo_ros_camera" filename="libgazebo_ros_camera.so">
-                <namespace>/sensors/cam</namespace>
-                <frame_name>camera_1</frame_name>
+                <namespace>head_camera/rgb</namespace>
+                <frame_name>head_camera_frame</frame_name>
             </plugin>
         </sensor>
     </gazebo>
-        <gazebo reference="wrist_camera_v1_1">
+    <gazebo reference="head_camera_frame">
+        <sensor type="depth" name="rgbd_camera">
+            <update_rate>30</update_rate>
+            <camera name="head_rgbd">
+            <horizontal_fov>1.0472</horizontal_fov>
+            <image>
+                <width>640</width>
+                <height>480</height>
+                <format>R8G8B8</format>
+            </image>
+            <clip>
+                <near>0.05</near>
+                <far>10.0</far>
+            </clip>
+            </camera>
+            <plugin name="gazebo_ros_depth_camera" filename="libgazebo_ros_camera.so">
+                <namespace>/head_camera/depth</namespace>
+                <frame_name>head_camera_frame</frame_name>
+            </plugin>
+        </sensor>
+    </gazebo>
+        <gazebo reference="wrist_camera_frame">
         <sensor type="camera" name="rgb_camera">
             <update_rate>30</update_rate>
@@ -44,27 +65,6 @@
             </camera>
             <plugin name="gazebo_ros_camera" filename="libgazebo_ros_camera.so">
-                <namespace>/sensors/wrist_camera</namespace>
-                <frame_name>wrist_camera</frame_name>
-            </plugin>
-        </sensor>
-    </gazebo>
-    <gazebo reference="head_camera_1">
-        <sensor type="depth" name="rgbd_camera">
-            <update_rate>30</update_rate>
-            <camera name="head_rgbd">
-            <horizontal_fov>1.0472</horizontal_fov>
-            <image>
-                <width>640</width>
-                <height>480</height>
-                <format>R8G8B8</format>
-            </image>
-            <clip>
-                <near>0.05</near>
-                <far>10.0</far>
-            </clip>
-            </camera>
-            <plugin name="gazebo_ros_depth_camera" filename="libgazebo_ros_camera.so">
-                <namespace>/sensors/rgbd</namespace>
-                <frame_name>camera_1</frame_name>
+                <namespace>/wrist_camera_frame/rgb</namespace>
+                <frame_name>wrist_camera_frame</frame_name>
             </plugin>
         </sensor>
@@ -99,5 +99,5 @@
         </sensor>
     </gazebo>
-    <gazebo reference="lidar_1">
+    <gazebo reference="lidar_frame">
         <sensor name="lidar" type="ray">
             <always_on>true</always_on>
@@ -107,8 +107,6 @@
             <scan>
                 <horizontal>
-                <samples>640</samples>
+                <samples>128</samples>
                 <resolution>1.000000</resolution>
-                <min_angle>-0.7955</min_angle>   <!-- -91.2/2 degrees -->
-                <max_angle>0.7955</max_angle>    <!-- +91.2/2 degrees -->
                 </horizontal>
             </scan>
@@ -129,5 +127,5 @@
             </ros>
             <output_type>sensor_msgs/LaserScan</output_type>
-            <frame_name>lidar_link</frame_name>
+            <frame_name>lidar_frame</frame_name>
             </plugin>
         </sensor>

Commit message: patched ros_control for tower

File: ros/src/leremix_description/urdf/LeRemix.xacro (robot description, xacro)
@@ -1339,5 +1339,5 @@
 </link>
 <joint name="head_camera_frame_joint" type="fixed">
-  <origin xyz="0.020 0.0 0.015" rpy="0 0 0"/>  <!-- Adjust to front center -->
+  <origin xyz="0.020 -0.022 0.0025" rpy="0 0 0"/>  <!-- Moved left 22mm, down 12.5mm -->
   <parent link="head_camera_1"/>
   <child link="head_camera_frame"/>
@@ -1347,5 +1347,5 @@
 </link>
 <joint name="wrist_camera_frame_joint" type="fixed">
-  <origin xyz="0.015 0.0 0.010" rpy="0 0 0"/>  <!-- Adjust to front center -->
+  <origin xyz="0.027 -0.012 0.010" rpy="3.14159 0 0"/>  <!-- Moved +12mm X, -12mm Y, rotated 180° around X -->
   <parent link="wrist_camera_v1_1"/>
   <child link="wrist_camera_frame"/>
@@ -1355,62 +1355,7 @@
 </link>
 <joint name="lidar_frame_joint" type="fixed">
-  <origin xyz="0.025 0.0 0.020" rpy="0 0 0"/>  <!-- Adjust to front center -->
+  <origin xyz="0.025 -0.0278 0.020" rpy="0 0 0"/>  <!-- Moved left by 27.8mm -->
   <parent link="lidar_1"/>
   <child link="lidar_frame"/>
 </joint>
-<!-- ros2_control hardware interface
-<ros2_control name="leremix_hardware" type="system">
-  <hardware>
-    <plugin>leremix_control_plugin/Esp32SystemTopic</plugin>
-    <param name="base_cmd_topic">/esp32/base_cmd</param>
-    <param name="arm_cmd_topic">/esp32/arm_cmd</param>
-    <param name="head_cmd_topic">/esp32/head_cmd</param>
-    <param name="state_topic">/esp32/joint_states</param>
-    <param name="publish_if_unchanged">true</param>
-  </hardware>
-  <joint name="back_motor_rotation">
-    <command_interface name="velocity"/>
-    <state_interface name="position"/>
-    <state_interface name="velocity"/>
-  </joint>
-  <joint name="left_motor_rotation">
-    <command_interface name="velocity"/>
-    <state_interface name="position"/>
-    <state_interface name="velocity"/>
-  </joint>
-  <joint name="right_motor_rotation">
-    <command_interface name="velocity"/>
-    <state_interface name="position"/>
-    <state_interface name="velocity"/>
-  </joint>
-  <joint name="1">
-    <command_interface name="position"/>
-    <state_interface name="position"/>
-  </joint>
-  <joint name="2">
-    <command_interface name="position"/>
-    <state_interface name="position"/>
-  </joint>
-  <joint name="3">
-    <command_interface name="position"/>
-    <state_interface name="position"/>
-  </joint>
-  <joint name="4">
-    <command_interface name="position"/>
-    <state_interface name="position"/>
-  </joint>
-  <joint name="5">
-    <command_interface name="position"/>
-    <state_interface name="position"/>
-  </joint>
-  <joint name="6">
-    <command_interface name="position"/>
-    <state_interface name="position"/>
-  </joint>
-  <joint name="camera_tilt">
-    <command_interface name="position"/>
-    <state_interface name="position"/>
-  </joint>
-</ros2_control>
--->
 </robot>
