Commit message: upgraded to foxy, added slam

File: ros/src/leremix_description/urdf/LeRemix.xacro (robot description, xacro)
@@ -5,4 +5,12 @@
 <link name="base_link">
 </link>
+    <!-- BASE_FOOTPRINT LINK -->
+    <joint name="base_footprint_joint" type="fixed">
+        <parent link="base_link"/>
+        <child link="base_footprint"/>
+        <origin xyz="0 0 0" rpy="0 0 0"/>
+    </joint>
+    <link name="base_footprint">
+    </link>
 <!-- Fixed joint to actual base -->
 <joint name="robot_base_joint" type="fixed">
@@ -20,5 +28,5 @@
     <origin xyz="0 0 0" rpy="0 0 0"/>
     <geometry>
-      <mesh filename="file://$(find leremix_description)/meshes/base_link.stl" scale="0.001 0.001 0.001"/>
+      <mesh filename="package://leremix_description/meshes/base_link.stl" scale="0.001 0.001 0.001"/>
     </geometry>
     <material name="Gazebo/DarkGrey"/>
@@ -27,5 +35,5 @@
     <origin xyz="0 0 0" rpy="0 0 0"/>
     <geometry>
-      <mesh filename="file://$(find leremix_description)/meshes/base_link.stl" scale="0.001 0.001 0.001"/>
+      <mesh filename="package://leremix_description/meshes/base_link.stl" scale="0.001 0.001 0.001"/>
     </geometry>
   </collision>
@@ -40,5 +48,5 @@
     <origin xyz="-0.050662 0.004002 -0.083133" rpy="0 0 0"/>
     <geometry>
-      <mesh filename="file://$(find leremix_description)/meshes/arm_base_rotation_servo_1.stl" scale="0.001 0.001 0.001"/>
+      <mesh filename="package://leremix_description/meshes/arm_base_rotation_servo_1.stl" scale="0.001 0.001 0.001"/>
     </geometry>
     <material name="Gazebo/DarkGrey"/>
@@ -47,5 +55,5 @@
     <origin xyz="-0.050662 0.004002 -0.083133" rpy="0 0 0"/>
     <geometry>
-      <mesh filename="file://$(find leremix_description)/meshes/arm_base_rotation_servo_1.stl" scale="0.001 0.001 0.001"/>
+      <mesh filename="package://leremix_description/meshes/arm_base_rotation_servo_1.stl" scale="0.001 0.001 0.001"/>
     </geometry>
   </collision>
@@ -60,5 +68,5 @@
     <origin xyz="-0.083462 -0.006248 -0.117733" rpy="0 0 0"/>
     <geometry>
-      <mesh filename="file://$(find leremix_description)/meshes/arm_base_rotation_link_1.stl" scale="0.001 0.001 0.001"/>
+      <mesh filename="package://leremix_description/meshes/arm_base_rotation_link_1.stl" scale="0.001 0.001 0.001"/>
     </geometry>
     <material name="Gazebo/DarkGrey"/>
@@ -67,5 +75,5 @@
     <origin xyz="-0.083462 -0.006248 -0.117733" rpy="0 0 0"/>
     <geometry>
-      <mesh filename="file://$(find leremix_description)/meshes/arm_base_rotation_link_1.stl" scale="0.001 0.001 0.001"/>
+      <mesh filename="package://leremix_description/meshes/arm_base_rotation_link_1.stl" scale="0.001 0.001 0.001"/>
     </geometry>
   </collision>
@@ -80,5 +88,5 @@
     <origin xyz="-0.124312 0.016752 -0.140933" rpy="0 0 0"/>
     <geometry>
-      <mesh filename="file://$(find leremix_description)/meshes/arm_base_rotation_link_cover_1.stl" scale="0.001 0.001 0.001"/>
+      <mesh filename="package://leremix_description/meshes/arm_base_rotation_link_cover_1.stl" scale="0.001 0.001 0.001"/>
     </geometry>
     <material name="Gazebo/DarkGrey"/>
@@ -87,5 +95,5 @@
     <origin xyz="-0.124312 0.016752 -0.140933" rpy="0 0 0"/>
     <geometry>
-      <mesh filename="file://$(find leremix_description)/meshes/arm_base_rotation_link_cover_1.stl" scale="0.001 0.001 0.001"/>
+      <mesh filename="package://leremix_description/meshes/arm_base_rotation_link_cover_1.stl" scale="0.001 0.001 0.001"/>
     </geometry>
   </collision>
@@ -100,5 +108,5 @@
     <origin xyz="-0.124312 -0.022548 -0.137133" rpy="0 0 0"/>
     <geometry>
-      <mesh filename="file://$(find leremix_description)/meshes/arm_shoulder_servo_1.stl" scale="0.001 0.001 0.001"/>
+      <mesh filename="package://leremix_description/meshes/arm_shoulder_servo_1.stl" scale="0.001 0.001 0.001"/>
     </geometry>
     <material name="Gazebo/DarkGrey"/>
@@ -107,5 +115,5 @@
     <origin xyz="-0.124312 -0.022548 -0.137133" rpy="0 0 0"/>
     <geometry>
-      <mesh filename="file://$(find leremix_description)/meshes/arm_shoulder_servo_1.stl" scale="0.001 0.001 0.001"/>
+      <mesh filename="package://leremix_description/meshes/arm_shoulder_servo_1.stl" scale="0.001 0.001 0.001"/>
     </geometry>
   </collision>
@@ -120,5 +128,5 @@
     <origin xyz="-0.114062 0.012052 -0.169933" rpy="0 0 0"/>
     <geometry>
-      <mesh filename="file://$(find leremix_description)/meshes/arm_shoulder_link_1.stl" scale="0.001 0.001 0.001"/>
+      <mesh filename="package://leremix_description/meshes/arm_shoulder_link_1.stl" scale="0.001 0.001 0.001"/>
     </geometry>
     <material name="Gazebo/DarkGrey"/>
@@ -127,5 +135,5 @@
     <origin xyz="-0.114062 0.012052 -0.169933" rpy="0 0 0"/>
     <geometry>
-      <mesh filename="file://$(find leremix_description)/meshes/arm_shoulder_link_1.stl" scale="0.001 0.001 0.001"/>
+      <mesh filename="package://leremix_description/meshes/arm_shoulder_link_1.stl" scale="0.001 0.001 0.001"/>
     </geometry>
   </collision>
@@ -140,5 +148,5 @@
     <origin xyz="-0.016471 -0.024048 -0.138814" rpy="0 0 0"/>
     <geometry>
-      <mesh filename="file://$(find leremix_description)/meshes/arm_elbow_servo_1.stl" scale="0.001 0.001 0.001"/>
+      <mesh filename="package://leremix_description/meshes/arm_elbow_servo_1.stl" scale="0.001 0.001 0.001"/>
     </geometry>
     <material name="Gazebo/DarkGrey"/>
@@ -147,5 +155,5 @@
     <origin xyz="-0.016471 -0.024048 -0.138814" rpy="0 0 0"/>
     <geometry>
-      <mesh filename="file://$(find leremix_description)/meshes/arm_elbow_servo_1.stl" scale="0.001 0.001 0.001"/>
+      <mesh filename="package://leremix_description/meshes/arm_elbow_servo_1.stl" scale="0.001 0.001 0.001"/>
     </geometry>
   </collision>
@@ -160,5 +168,5 @@
     <origin xyz="0.001919 0.010552 -0.167844" rpy="0 0 0"/>
     <geometry>
-      <mesh filename="file://$(find leremix_description)/meshes/arm_elbow_link_1.stl" scale="0.001 0.001 0.001"/>
+      <mesh filename="package://leremix_description/meshes/arm_elbow_link_1.stl" scale="0.001 0.001 0.001"/>
     </geometry>
     <material name="Gazebo/DarkGrey"/>
@@ -167,5 +175,5 @@
     <origin xyz="0.001919 0.010552 -0.167844" rpy="0 0 0"/>
     <geometry>
-      <mesh filename="file://$(find leremix_description)/meshes/arm_elbow_link_1.stl" scale="0.001 0.001 0.001"/>
+      <mesh filename="package://leremix_description/meshes/arm_elbow_link_1.stl" scale="0.001 0.001 0.001"/>
     </geometry>
   </collision>
@@ -180,5 +188,5 @@
     <origin xyz="-0.089679 -0.025548 -0.217624" rpy="0 0 0"/>
     <geometry>
-      <mesh filename="file://$(find leremix_description)/meshes/arm_wrist_tilt_servo_1.stl" scale="0.001 0.001 0.001"/>
+      <mesh filename="package://leremix_description/meshes/arm_wrist_tilt_servo_1.stl" scale="0.001 0.001 0.001"/>
     </geometry>
     <material name="Gazebo/DarkGrey"/>
@@ -187,5 +195,5 @@
     <origin xyz="-0.089679 -0.025548 -0.217624" rpy="0 0 0"/>
     <geometry>
-      <mesh filename="file://$(find leremix_description)/meshes/arm_wrist_tilt_servo_1.stl" scale="0.001 0.001 0.001"/>
+      <mesh filename="package://leremix_description/meshes/arm_wrist_tilt_servo_1.stl" scale="0.001 0.001 0.001"/>
     </geometry>
   </collision>
@@ -200,5 +208,5 @@
     <origin xyz="-0.124014 0.009052 -0.216213" rpy="0 0 0"/>
     <geometry>
-      <mesh filename="file://$(find leremix_description)/meshes/arm_wrist_link_1.stl" scale="0.001 0.001 0.001"/>
+      <mesh filename="package://leremix_description/meshes/arm_wrist_link_1.stl" scale="0.001 0.001 0.001"/>
     </geometry>
     <material name="Gazebo/DarkGrey"/>
@@ -207,5 +215,5 @@
     <origin xyz="-0.124014 0.009052 -0.216213" rpy="0 0 0"/>
     <geometry>
-      <mesh filename="file://$(find leremix_description)/meshes/arm_wrist_link_1.stl" scale="0.001 0.001 0.001"/>
+      <mesh filename="package://leremix_description/meshes/arm_wrist_link_1.stl" scale="0.001 0.001 0.001"/>
     </geometry>
   </collision>
@@ -220,5 +228,5 @@
     <origin xyz="-0.161703 0.017952 -0.170568" rpy="0 0 0"/>
     <geometry>
-      <mesh filename="file://$(find leremix_description)/meshes/arm_wrist_roll_servo_1.stl" scale="0.001 0.001 0.001"/>
+      <mesh filename="package://leremix_description/meshes/arm_wrist_roll_servo_1.stl" scale="0.001 0.001 0.001"/>
     </geometry>
     <material name="Gazebo/DarkGrey"/>
@@ -227,5 +235,5 @@
     <origin xyz="-0.161703 0.017952 -0.170568" rpy="0 0 0"/>
     <geometry>
-      <mesh filename="file://$(find leremix_description)/meshes/arm_wrist_roll_servo_1.stl" scale="0.001 0.001 0.001"/>
+      <mesh filename="package://leremix_description/meshes/arm_wrist_roll_servo_1.stl" scale="0.001 0.001 0.001"/>
     </geometry>
   </collision>
@@ -240,5 +248,5 @@
     <origin xyz="-0.15417 -0.011048 -0.163073" rpy="0 0 0"/>
     <geometry>
-      <mesh filename="file://$(find leremix_description)/meshes/arm_gripper_1.stl" scale="0.001 0.001 0.001"/>
+      <mesh filename="package://leremix_description/meshes/arm_gripper_1.stl" scale="0.001 0.001 0.001"/>
     </geometry>
     <material name="Gazebo/DarkGrey"/>
@@ -247,5 +255,5 @@
     <origin xyz="-0.15417 -0.011048 -0.163073" rpy="0 0 0"/>
     <geometry>
-      <mesh filename="file://$(find leremix_description)/meshes/arm_gripper_1.stl" scale="0.001 0.001 0.001"/>
+      <mesh filename="package://leremix_description/meshes/arm_gripper_1.stl" scale="0.001 0.001 0.001"/>
     </geometry>
   </collision>
@@ -260,5 +268,5 @@
     <origin xyz="-0.173846 0.00275 -0.159436" rpy="0 0 0"/>
     <geometry>
-      <mesh filename="file://$(find leremix_description)/meshes/arm_gripper_servo_1.stl" scale="0.001 0.001 0.001"/>
+      <mesh filename="package://leremix_description/meshes/arm_gripper_servo_1.stl" scale="0.001 0.001 0.001"/>
     </geometry>
     <material name="Gazebo/DarkGrey"/>
@@ -267,5 +275,5 @@
     <origin xyz="-0.173846 0.00275 -0.159436" rpy="0 0 0"/>
     <geometry>
-      <mesh filename="file://$(find leremix_description)/meshes/arm_gripper_servo_1.stl" scale="0.001 0.001 0.001"/>
+      <mesh filename="package://leremix_description/meshes/arm_gripper_servo_1.stl" scale="0.001 0.001 0.001"/>
     </geometry>
   </collision>
@@ -280,5 +288,5 @@
     <origin xyz="-0.150306 -0.03177 -0.134291" rpy="0 0 0"/>
     <geometry>
-      <mesh filename="file://$(find leremix_description)/meshes/arm_jaw_1.stl" scale="0.001 0.001 0.001"/>
+      <mesh filename="package://leremix_description/meshes/arm_jaw_1.stl" scale="0.001 0.001 0.001"/>
     </geometry>
     <material name="Gazebo/DarkGrey"/>
@@ -287,5 +295,5 @@
     <origin xyz="-0.150306 -0.03177 -0.134291" rpy="0 0 0"/>
     <geometry>
-      <mesh filename="file://$(find leremix_description)/meshes/arm_jaw_1.stl" scale="0.001 0.001 0.001"/>
+      <mesh filename="package://leremix_description/meshes/arm_jaw_1.stl" scale="0.001 0.001 0.001"/>
     </geometry>
   </collision>
@@ -300,5 +308,5 @@
     <origin xyz="-0.028994 0.073033 -0.002833" rpy="0 0 0"/>
     <geometry>
-      <mesh filename="file://$(find leremix_description)/meshes/right_servo_mount_1.stl" scale="0.001 0.001 0.001"/>
+      <mesh filename="package://leremix_description/meshes/right_servo_mount_1.stl" scale="0.001 0.001 0.001"/>
     </geometry>
     <material name="Gazebo/DarkGrey"/>
@@ -307,5 +315,5 @@
     <origin xyz="-0.028994 0.073033 -0.002833" rpy="0 0 0"/>
     <geometry>
-      <mesh filename="file://$(find leremix_description)/meshes/right_servo_mount_1.stl" scale="0.001 0.001 0.001"/>
+      <mesh filename="package://leremix_description/meshes/right_servo_mount_1.stl" scale="0.001 0.001 0.001"/>
     </geometry>
   </collision>
@@ -320,5 +328,5 @@
     <origin xyz="-0.034659 0.063359 -0.021333" rpy="0 0 0"/>
     <geometry>
-      <mesh filename="file://$(find leremix_description)/meshes/right_servo_1.stl" scale="0.001 0.001 0.001"/>
+      <mesh filename="package://leremix_description/meshes/right_servo_1.stl" scale="0.001 0.001 0.001"/>
     </geometry>
     <material name="Gazebo/DarkGrey"/>
@@ -327,5 +335,5 @@
     <origin xyz="-0.034659 0.063359 -0.021333" rpy="0 0 0"/>
     <geometry>
-      <mesh filename="file://$(find leremix_description)/meshes/right_servo_1.stl" scale="0.001 0.001 0.001"/>
+      <mesh filename="package://leremix_description/meshes/right_servo_1.stl" scale="0.001 0.001 0.001"/>
     </geometry>
   </collision>
@@ -340,5 +348,5 @@
     <origin xyz="-0.060348 0.087326 -0.013051" rpy="0 0 0"/>
     <geometry>
-      <mesh filename="file://$(find leremix_description)/meshes/right_wheel_mount_1.stl" scale="0.001 0.001 0.001"/>
+      <mesh filename="package://leremix_description/meshes/right_wheel_mount_1.stl" scale="0.001 0.001 0.001"/>
     </geometry>
     <material name="Gazebo/DarkGrey"/>
@@ -347,5 +355,5 @@
     <origin xyz="-0.060348 0.087326 -0.013051" rpy="0 0 0"/>
     <geometry>
-      <mesh filename="file://$(find leremix_description)/meshes/right_wheel_mount_1.stl" scale="0.001 0.001 0.001"/>
+      <mesh filename="package://leremix_description/meshes/right_wheel_mount_1.stl" scale="0.001 0.001 0.001"/>
     </geometry>
   </collision>
@@ -360,5 +368,5 @@
     <origin xyz="0.093686 0.013751 -0.002833" rpy="0 0 0"/>
     <geometry>
-      <mesh filename="file://$(find leremix_description)/meshes/back_servo_mount_1.stl" scale="0.001 0.001 0.001"/>
+      <mesh filename="package://leremix_description/meshes/back_servo_mount_1.stl" scale="0.001 0.001 0.001"/>
     </geometry>
     <material name="Gazebo/DarkGrey"/>
@@ -367,5 +375,5 @@
     <origin xyz="0.093686 0.013751 -0.002833" rpy="0 0 0"/>
     <geometry>
-      <mesh filename="file://$(find leremix_description)/meshes/back_servo_mount_1.stl" scale="0.001 0.001 0.001"/>
+      <mesh filename="package://leremix_description/meshes/back_servo_mount_1.stl" scale="0.001 0.001 0.001"/>
     </geometry>
   </collision>
@@ -380,5 +388,5 @@
     <origin xyz="-0.038994 -0.102851 -0.002833" rpy="0 0 0"/>
     <geometry>
-      <mesh filename="file://$(find leremix_description)/meshes/left_servo_mount_1.stl" scale="0.001 0.001 0.001"/>
+      <mesh filename="package://leremix_description/meshes/left_servo_mount_1.stl" scale="0.001 0.001 0.001"/>
     </geometry>
     <material name="Gazebo/DarkGrey"/>
@@ -387,5 +395,5 @@
     <origin xyz="-0.038994 -0.102851 -0.002833" rpy="0 0 0"/>
     <geometry>
-      <mesh filename="file://$(find leremix_description)/meshes/left_servo_mount_1.stl" scale="0.001 0.001 0.001"/>
+      <mesh filename="package://leremix_description/meshes/left_servo_mount_1.stl" scale="0.001 0.001 0.001"/>
     </geometry>
   </collision>
@@ -400,5 +408,5 @@
     <origin xyz="0.068141 -0.016505 -0.045832" rpy="0 0 0"/>
     <geometry>
-      <mesh filename="file://$(find leremix_description)/meshes/back_servo_1.stl" scale="0.001 0.001 0.001"/>
+      <mesh filename="package://leremix_description/meshes/back_servo_1.stl" scale="0.001 0.001 0.001"/>
     </geometry>
     <material name="Gazebo/DarkGrey"/>
@@ -407,5 +415,5 @@
     <origin xyz="0.068141 -0.016505 -0.045832" rpy="0 0 0"/>
     <geometry>
-      <mesh filename="file://$(find leremix_description)/meshes/back_servo_1.stl" scale="0.001 0.001 0.001"/>
+      <mesh filename="package://leremix_description/meshes/back_servo_1.stl" scale="0.001 0.001 0.001"/>
     </geometry>
   </collision>
@@ -420,5 +428,5 @@
     <origin xyz="-0.063935 0.09354 -0.013051" rpy="0 0 0"/>
     <geometry>
-      <mesh filename="file://$(find leremix_description)/meshes/right_wheel_1.stl" scale="0.001 0.001 0.001"/>
+      <mesh filename="package://leremix_description/meshes/right_wheel_1.stl" scale="0.001 0.001 0.001"/>
     </geometry>
     <material name="Gazebo/DarkGrey"/>
@@ -427,5 +435,5 @@
     <origin xyz="-0.063935 0.09354 -0.013051" rpy="0 0 0"/>
     <geometry>
-      <mesh filename="file://$(find leremix_description)/meshes/right_wheel_1.stl" scale="0.001 0.001 0.001"/>
+      <mesh filename="package://leremix_description/meshes/right_wheel_1.stl" scale="0.001 0.001 0.001"/>
     </geometry>
   </collision>
@@ -440,5 +448,5 @@
     <origin xyz="0.101741 -0.006255 -0.013032" rpy="0 0 0"/>
     <geometry>
-      <mesh filename="file://$(find leremix_description)/meshes/back_wheel_mount_1.stl" scale="0.001 0.001 0.001"/>
+      <mesh filename="package://leremix_description/meshes/back_wheel_mount_1.stl" scale="0.001 0.001 0.001"/>
     </geometry>
     <material name="Gazebo/DarkGrey"/>
@@ -447,5 +455,5 @@
     <origin xyz="0.101741 -0.006255 -0.013032" rpy="0 0 0"/>
     <geometry>
-      <mesh filename="file://$(find leremix_description)/meshes/back_wheel_mount_1.stl" scale="0.001 0.001 0.001"/>
+      <mesh filename="package://leremix_description/meshes/back_wheel_mount_1.stl" scale="0.001 0.001 0.001"/>
     </geometry>
   </collision>
@@ -460,5 +468,5 @@
     <origin xyz="0.108916 -0.006255 -0.013032" rpy="0 0 0"/>
     <geometry>
-      <mesh filename="file://$(find leremix_description)/meshes/back_wheel_1.stl" scale="0.001 0.001 0.001"/>
+      <mesh filename="package://leremix_description/meshes/back_wheel_1.stl" scale="0.001 0.001 0.001"/>
     </geometry>
     <material name="Gazebo/DarkGrey"/>
@@ -467,5 +475,5 @@
     <origin xyz="0.108916 -0.006255 -0.013032" rpy="0 0 0"/>
     <geometry>
-      <mesh filename="file://$(find leremix_description)/meshes/back_wheel_1.stl" scale="0.001 0.001 0.001"/>
+      <mesh filename="package://leremix_description/meshes/back_wheel_1.stl" scale="0.001 0.001 0.001"/>
     </geometry>
   </collision>
@@ -480,5 +488,5 @@
     <origin xyz="-0.034669 -0.07585 -0.045832" rpy="0 0 0"/>
     <geometry>
-      <mesh filename="file://$(find leremix_description)/meshes/left_servo_1.stl" scale="0.001 0.001 0.001"/>
+      <mesh filename="package://leremix_description/meshes/left_servo_1.stl" scale="0.001 0.001 0.001"/>
     </geometry>
     <material name="Gazebo/DarkGrey"/>
@@ -487,5 +495,5 @@
     <origin xyz="-0.034669 -0.07585 -0.045832" rpy="0 0 0"/>
     <geometry>
-      <mesh filename="file://$(find leremix_description)/meshes/left_servo_1.stl" scale="0.001 0.001 0.001"/>
+      <mesh filename="package://leremix_description/meshes/left_servo_1.stl" scale="0.001 0.001 0.001"/>
     </geometry>
   </collision>
@@ -500,5 +508,5 @@
     <origin xyz="-0.060298 -0.099852 -0.013014" rpy="0 0 0"/>
     <geometry>
-      <mesh filename="file://$(find leremix_description)/meshes/left_wheel_mount_1.stl" scale="0.001 0.001 0.001"/>
+      <mesh filename="package://leremix_description/meshes/left_wheel_mount_1.stl" scale="0.001 0.001 0.001"/>
     </geometry>
     <material name="Gazebo/DarkGrey"/>
@@ -507,5 +515,5 @@
     <origin xyz="-0.060298 -0.099852 -0.013014" rpy="0 0 0"/>
     <geometry>
-      <mesh filename="file://$(find leremix_description)/meshes/left_wheel_mount_1.stl" scale="0.001 0.001 0.001"/>
+      <mesh filename="package://leremix_description/meshes/left_wheel_mount_1.stl" scale="0.001 0.001 0.001"/>
     </geometry>
   </collision>
@@ -520,5 +528,5 @@
     <origin xyz="-0.063885 -0.106065 -0.013014" rpy="0 0 0"/>
     <geometry>
-      <mesh filename="file://$(find leremix_description)/meshes/left_wheel_1.stl" scale="0.001 0.001 0.001"/>
+      <mesh filename="package://leremix_description/meshes/left_wheel_1.stl" scale="0.001 0.001 0.001"/>
     </geometry>
     <material name="Gazebo/DarkGrey"/>
@@ -527,5 +535,5 @@
     <origin xyz="-0.063885 -0.106065 -0.013014" rpy="0 0 0"/>
     <geometry>
-      <mesh filename="file://$(find leremix_description)/meshes/left_wheel_1.stl" scale="0.001 0.001 0.001"/>
+      <mesh filename="package://leremix_description/meshes/left_wheel_1.stl" scale="0.001 0.001 0.001"/>
     </geometry>
   </collision>
@@ -540,5 +548,5 @@
     <origin xyz="0.015686 0.039888 -0.067333" rpy="0 0 0"/>
     <geometry>
-      <mesh filename="file://$(find leremix_description)/meshes/orin_1.stl" scale="0.001 0.001 0.001"/>
+      <mesh filename="package://leremix_description/meshes/orin_1.stl" scale="0.001 0.001 0.001"/>
     </geometry>
     <material name="Gazebo/DarkGrey"/>
@@ -547,5 +555,5 @@
     <origin xyz="0.015686 0.039888 -0.067333" rpy="0 0 0"/>
     <geometry>
-      <mesh filename="file://$(find leremix_description)/meshes/orin_1.stl" scale="0.001 0.001 0.001"/>
+      <mesh filename="package://leremix_description/meshes/orin_1.stl" scale="0.001 0.001 0.001"/>
     </geometry>
   </collision>
@@ -560,5 +568,5 @@
     <origin xyz="0.093686 0.033751 -0.055333" rpy="0 0 0"/>
     <geometry>
-      <mesh filename="file://$(find leremix_description)/meshes/orin_mount_1.stl" scale="0.001 0.001 0.001"/>
+      <mesh filename="package://leremix_description/meshes/orin_mount_1.stl" scale="0.001 0.001 0.001"/>
     </geometry>
     <material name="Gazebo/DarkGrey"/>
@@ -567,5 +575,5 @@
     <origin xyz="0.093686 0.033751 -0.055333" rpy="0 0 0"/>
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