Commit message: updates on harmonic simulation

File: ros/src/leremix_description/urdf/LeRemix.xacro (robot description, xacro)
@@ -22,5 +22,5 @@
   <inertial>
     <origin xyz="5.866413998148801e-05 0.0062819967824381704 0.001416599330144379" rpy="0 0 0"/>
-    <mass value="3.24"/>  <!-- base(440g) + battery(800g) -->
+    <mass value="6.0"/>  <!-- increased for simulation stability -->
     <inertia ixx="0.012" iyy="0.015" izz="0.020" ixy="-3.5e-06" iyz="0.0" ixz="0.0"/>
   </inertial>
@@ -433,7 +433,7 @@
   </visual>
   <collision>
-    <origin xyz="-0.063935 0.09354 -0.013051" rpy="0 0 0"/>
-    <geometry>
-      <mesh filename="package://leremix_description/meshes/right_wheel_1.stl" scale="0.001 0.001 0.001"/>
+    <origin xyz="0.008 -0.013 0" rpy="0 1.5708 2.0944"/>
+    <geometry>
+      <cylinder radius="0.05" length="0.025"/>
     </geometry>
   </collision>
@@ -473,7 +473,7 @@
   </visual>
   <collision>
-    <origin xyz="0.108916 -0.006255 -0.013032" rpy="0 0 0"/>
-    <geometry>
-      <mesh filename="package://leremix_description/meshes/back_wheel_1.stl" scale="0.001 0.001 0.001"/>
+    <origin xyz="-0.015 0 0" rpy="0 1.5708 0"/>
+    <geometry>
+      <cylinder radius="0.05" length="0.025"/>
     </geometry>
   </collision>
@@ -533,7 +533,7 @@
   </visual>
   <collision>
-    <origin xyz="-0.063885 -0.106065 -0.013014" rpy="0 0 0"/>
-    <geometry>
-      <mesh filename="package://leremix_description/meshes/left_wheel_1.stl" scale="0.001 0.001 0.001"/>
+    <origin xyz="0.008 0.013 0" rpy="0 1.5708 -2.0944"/>
+    <geometry>
+      <cylinder radius="0.05" length="0.025"/>
     </geometry>
   </collision>
@@ -1157,4 +1157,5 @@
   <child link="right_wheel_mount_1"/>
   <axis xyz="-0.5 0.866025 -0.0"/>
+  <dynamics damping="0.01" friction="0.005"/>
 </joint>
 <joint name="Rigid 79" type="fixed">
@@ -1183,4 +1184,5 @@
   <child link="back_wheel_mount_1"/>
   <axis xyz="-1.0 -0.0 -0.0"/>
+  <dynamics damping="0.01" friction="0.005"/>
 </joint>
 <joint name="Rigid 85" type="fixed">
@@ -1199,4 +1201,5 @@
   <child link="left_wheel_mount_1"/>
   <axis xyz="-0.5 -0.866025 -0.0"/>
+  <dynamics damping="0.01" friction="0.005"/>
 </joint>
 <joint name="Rigid 88" type="fixed">

File: ros/src/leremix_gazebo/urdf/gazebo_configs.xacro (robot description, xacro)
@@ -1,23 +1,4 @@
 <robot xmlns:xacro="http://www.ros.org/wiki/xacro" name="LeRemix">
-<physics type="ode" default="true">
-  <max_step_size>0.001</max_step_size>
-  <real_time_update_rate>1000</real_time_update_rate>
-   <ode>
-    <solver type="quick" iters="150" sor="1.3"/>
-    <constraints cfm="0.0" erp="0.2"
-      contact_max_correcting_vel="0.5"
-      contact_surface_layer="0.001"/>
-  </ode>
-</physics>
-<physics type="ode">
-  <max_step_size>0.001</max_step_size>
-  <real_time_update_rate>1000</real_time_update_rate>
-  <ode>
-    <solver type="quick" iters="150" sor="1.3"/>
-    <constraints cfm="0.0" erp="0.2"
-      contact_max_correcting_vel="0.5"
-      contact_surface_layer="0.001"/>
-  </ode>
-</physics>
+<!-- Physics parameters are configured in world file for Gazebo Harmonic -->
 <gazebo reference="base_link">
   <material>Gazebo/FlatBlack</material>
@@ -321,7 +302,7 @@
   <fdir1>-0.866025 -0.5 0</fdir1>
   <slip1>0.0</slip1>
-  <slip2>0.01</slip2>
-  <kp>1.8e6</kp>
-  <kd>3.5</kd>
+  <slip2>0.1</slip2>
+  <kp>1e5</kp>
+  <kd>100</kd>
 </gazebo>
 <gazebo reference="back_wheel_1">
@@ -330,7 +311,7 @@
   <fdir1>0 -1 0</fdir1>
   <slip1>0.0</slip1>
-  <slip2>0.01</slip2>
-  <kp>1.8e6</kp>
-  <kd>3.5</kd>
+  <slip2>0.1</slip2>
+  <kp>1e5</kp>
+  <kd>100</kd>
 </gazebo>
 <gazebo reference="left_wheel_1">
@@ -339,7 +320,7 @@
   <fdir1>0.866025 -0.5 0</fdir1>
   <slip1>0.0</slip1>
-  <slip2>0.01</slip2>
-  <kp>1.8e6</kp>
-  <kd>3.5</kd>
+  <slip2>0.1</slip2>
+  <kp>1e5</kp>
+  <kd>100</kd>
 </gazebo>
 <gazebo reference="lidar_1">

File: ros/src/leremix_gazebo/urdf/gazebo_interfaces.xacro (robot description, xacro)
@@ -3,5 +3,5 @@
   <ros2_control name="GazeboSystem" type="system">
         <hardware>
-            <plugin>gazebo_ros2_control/GazeboSystem</plugin>
+            <plugin>gz_ros2_control/GazeboSimSystem</plugin>
         </hardware>
         <joint name="wheel1_rotation">
